File: MasterShield.kicad_sch (KiCad schematic)
At the start: 31 parts, among them J1 Conn_01x08_Pin, J2 Conn_01x10_Pin, J3 Conn_01x06_Pin, J4 Conn_01x08_Pin, J5 RS485, J6 Screw_Terminal_01x08, Q1 S8050, U1 MAX485E, U2 BTS724G, U3 74LVC1G08GW

Commit message: ...
Parts:
- added TP1: RO, symbol Connector:TestPoint
- added TP2: DI, symbol Connector:TestPoint
- added TP3: ~{RE}, symbol Connector:TestPoint
- added TP4: DE, symbol Connector:TestPoint
Connections:
- net P0.00: now also TP1.1
- net P0.01: now also TP2.1
- net at R10.2, R11.2, R2.2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: now also TP3.1
- net at U1.3 (DE), U3.4: now also TP4.1
Changed lines of the file:
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@@
   (junction (at 127 74.93) (diameter 0) (color 0 0 0 0)
   )
+  (junction (at 92.71 57.15) (diameter 0) (color 0 0 0 0)
+  )
   (junction (at 204.47 39.37) (diameter 0) (color 0 0 0 0)
   )
@@
   (junction (at 204.47 25.4) (diameter 0) (color 0 0 0 0)
   )
+  (junction (at 104.14 52.07) (diameter 0) (color 0 0 0 0)
+  )
   (junction (at 222.25 68.58) (diameter 0) (color 0 0 0 0)
   )
@@
   (junction (at 99.06 53.34) (diameter 0) (color 0 0 0 0)
   )
+  (junction (at 109.22 63.5) (diameter 0) (color 0 0 0 0)
+  )
   (junction (at 99.06 49.53) (diameter 0) (color 0 0 0 0)
   )
   (junction (at 40.64 110.49) (diameter 0) (color 0 0 0 0)
+  )
+  (junction (at 102.87 49.53) (diameter 0) (color 0 0 0 0)
   )
   (no_connect (at 34.29 125.73))
@@
     (stroke (width 0) (type default))
   )
+  (wire (pts (xy 102.87 49.53) (xy 116.84 49.53))
+    (stroke (width 0) (type default))
+  )
   (wire (pts (xy 25.4 123.19) (xy 40.64 123.19))
     (stroke (width 0) (type default))
   )
-  (wire (pts (xy 109.22 52.07) (xy 99.06 52.07))
+  (wire (pts (xy 109.22 52.07) (xy 104.14 52.07))
     (stroke (width 0) (type default))
   )
@@
     (stroke (width 0) (type default))
   )
+  (wire (pts (xy 109.22 63.5) (xy 109.22 81.28))
+    (stroke (width 0) (type default))
+  )
   (wire (pts (xy 127 25.4) (xy 127 39.37))
     (stroke (width 0) (type default))
@@
     (stroke (width 0) (type default))
   )
-  (wire (pts (xy 99.06 49.53) (xy 116.84 49.53))
+  (wire (pts (xy 92.71 57.15) (xy 116.84 57.15))
+    (stroke (width 0) (type default))
+  )
+  (wire (pts (xy 99.06 49.53) (xy 102.87 49.53))
     (stroke (width 0) (type default))
   )
@@
     (stroke (width 0) (type default))
   )
-  (wire (pts (xy 109.22 81.28) (xy 109.22 54.61))
-    (stroke (width 0) (type default))
-  )
   (wire (pts (xy 143.51 64.77) (xy 151.13 64.77))
     (stroke (width 0) (type default))
@@
     (stroke (width 0) (type default))
   )
+  (wire (pts (xy 109.22 63.5) (xy 109.22 54.61))
+    (stroke (width 0) (type default))
+  )
   (wire (pts (xy 168.91 52.07) (xy 163.83 52.07))
     (stroke (width 0) (type default))
@@
     (stroke (width 0) (type default))
   )
+  (wire (pts (xy 104.14 52.07) (xy 99.06 52.07))
+    (stroke (width 0) (type default))
+  )
   (wire (pts (xy 25.4 59.69) (xy 36.83 59.69))
     (stroke (width 0) (type default))
@@
     (stroke (width 0) (type default))
   )
+  (wire (pts (xy 111.76 52.07) (xy 111.76 87.63))
+    (stroke (width 0) (type default))
+  )
   (wire (pts (xy 127 74.93) (xy 99.06 74.93))
     (stroke (width 0) (type default))
@@
     (stroke (width 0) (type default))
   )
-  (wire (pts (xy 88.9 57.15) (xy 116.84 57.15))
+  (wire (pts (xy 88.9 57.15) (xy 92.71 57.15))
     (stroke (width 0) (type default))
   )
@@
     (stroke (width 0) (type default))
   )
-  (wire (pts (xy 111.76 87.63) (xy 111.76 52.07))
-    (stroke (width 0) (type default))
-  )
   (wire (pts (xy 242.57 39.37) (xy 237.49 39.37))
     (stroke (width 0) (type default))
@@
   (label "TXD" (at 85.09 57.15 0) (fields_autoplaced)
     (effects (font (size 1.27 1.27)) (justify left bottom))
+  )
+  (symbol (lib_id "Connector:TestPoint") (at 92.71 57.15 180) (unit 1)
+    (in_bom yes) (on_board yes) (dnp no)
+    (property "Reference" "TP2" (at 93.98 58.42 0)
+      (effects (font (size 1.27 1.27)) (justify right))
+    )
+    (property "Value" "DI" (at 93.98 60.96 0)
+      (effects (font (size 1.27 1.27)) (justify right))
+    )
+    (property "Footprint" "" (at 87.63 57.15 0)
+      (effects (font (size 1.27 1.27)) hide)
+    )
+    (property "Datasheet" "~" (at 87.63 57.15 0)
+      (effects (font (size 1.27 1.27)) hide)
+    )
+    (pin "1")
+    (instances
+      (project "MasterShield"
+        (path "/16d5516d-cfb1-48ac-a57f-0957fae4baa5"
+          (reference "TP2") (unit 1)
+        )
+      )
+    )
   )
   (symbol (lib_id "power:GND") (at 222.25 74.93 0) (unit 1)
@@
     )
   )
+  (symbol (lib_id "Connector:TestPoint") (at 102.87 49.53 0) (unit 1)
+    (in_bom yes) (on_board yes) (dnp no) (fields_autoplaced)
+    (property "Reference" "TP1" (at 105.41 44.958 0)
+      (effects (font (size 1.27 1.27)) (justify left))
+    )
+    (property "Value" "RO" (at 105.41 47.498 0)
+      (effects (font (size 1.27 1.27)) (justify left))
+    )
+    (property "Footprint" "" (at 107.95 49.53 0)
+      (effects (font (size 1.27 1.27)) hide)
+    )
+    (property "Datasheet" "~" (at 107.95 49.53 0)
+      (effects (font (size 1.27 1.27)) hide)
+    )
+    (pin "1")
+    (instances
+      (project "MasterShield"
+        (path "/16d5516d-cfb1-48ac-a57f-0957fae4baa5"
+          (reference "TP1") (unit 1)
+        )
+      )
+    )
+  )
   (symbol (lib_id "power:GND") (at 121.92 93.98 90) (unit 1)
     (in_bom yes) (on_board yes) (dnp no) (fields_autoplaced)
@@
         (path "/16d5516d-cfb1-48ac-a57f-0957fae4baa5"
           (reference "J5") (unit 1)
+        )
+      )
+    )
+  )
+  (symbol (lib_id "Connector:TestPoint") (at 109.22 63.5 90) (unit 1)
+    (in_bom yes) (on_board yes) (dnp no)
+    (property "Reference" "TP4" (at 101.6 63.5 90)
+      (effects (font (size 1.27 1.27)) (justify right))
+    )
+    (property "Value" "DE" (at 104.14 60.96 90)
+      (effects (font (size 1.27 1.27)) (justify right))
+    )
+    (property "Footprint" "" (at 109.22 58.42 0)
+      (effects (font (size 1.27 1.27)) hide)
+    )
+    (property "Datasheet" "~" (at 109.22 58.42 0)
+      (effects (font (size 1.27 1.27)) hide)
+    )
+    (pin "1")
+    (instances
+      (project "MasterShield"
+        (path "/16d5516d-cfb1-48ac-a57f-0957fae4baa5"
+          (reference "TP4") (unit 1)
         )
       )
@@
         )
       )
+    )
+  )
+  (symbol (lib_id "Connector:TestPoint") (at 104.14 52.07 180) (unit 1)
+    (in_bom yes) (on_board yes) (dnp no)
+    (property "Reference" "TP3" (at 105.41 53.34 0)
+      (effects (font (size 1.27 1.27)) (justify right))
+    )
+    (property "Value" "~{RE}" (at 105.41 55.88 0)
+      (effects (font (size 1.27 1.27)) (justify right))
+    )
+    (property "Footprint" "" (at 99.06 52.07 0)
+      (effects (font (size 1.27 1.27)) hide)
+    )
+    (property "Datasheet" "~" (at 99.06 52.07 0)
+      (effects (font (size 1.27 1.27)) hide)
+    )
+    (pin "1")
+    (instances
+      (project "MasterShield"
+        (path "/16d5516d-cfb1-48ac-a57f-0957fae4baa5"
+          (reference "TP3") (unit 1)
+        )
+      )

Commit message: ...
Parts:
- added C4: 68uF, Capacitor_Tantalum_SMD:CP_EIA-7343-43_Kemet-X, symbol Device:C_Polarized
- added C5: 150uF, Capacitor_Tantalum_SMD:CP_EIA-7343-43_Kemet-X, symbol Device:C_Polarized
- added D3: B5817, Diode_SMD:D_SOD-323_HandSoldering, symbol Diode:1N5817
- added L1: 100uH, Inductor_SMD:L_12x12mm_H6mm, symbol Device:L
- added U4: LM2594M-5.0, Package_SO:SOIC-8_3.9x4.9mm_P1.27mm, symbol Regulator_Switching:LM2594M-5.0
- TP1, TP2, TP3, TP4: footprint (none) -> TestPoint:TestPoint_Pad_D2.0mm
Connections:
- net +12V: now also C4.1, U4.7 (VIN)
- net +5V: now also C5.1, L1.2, U4.4 (FB)
- net GND: now also C4.2, C5.2, D3.2 (A), U4.5 (~{ON}/OFF), U4.6 (GND)
- new net: D3.1 (K), L1.1, U4.8 (OUT)
- no-connect marks 1 -> 4

Commit message: ...
Parts:
- removed U4: LM2594M-5.0, Package_SO:SOIC-8_3.9x4.9mm_P1.27mm, symbol Regulator_Switching:LM2594M-5.0
- added U5: LM2596S-5, Package_TO_SOT_SMD:TO-263-5_TabPin3, symbol Regulator_Switching:LM2596S-5
- C4: value 68uF -> 680uF; footprint Capacitor_Tantalum_SMD:CP_EIA-7343-43_Kemet-X -> Capacitor_SMD:CP_Elec_10x10.5; LCSC https://www.lcsc.com/product-detail/Tantalum-Capacitors_KEM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 -> https://www.lcsc.com/product-detail/Aluminum-Electrolytic-C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
- C5: value 150uF -> 220uF; footprint Capacitor_Tantalum_SMD:CP_EIA-7343-43_Kemet-X -> Capacitor_Tantalum_SMD:CP_EIA-7343-15_Kemet-W_Pad2.25x2.55mm_HandSolder; LCSC https://www.lcsc.com/product-detail/Tantalum-Capacitors_Kyo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 -> https://www.lcsc.com/product-detail/Tantalum-Capacitors_KEM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
- D3: value B5817 -> SS53C; LCSCL (none) -> https://www.lcsc.com/product-detail/Schottky-Barrier-Diodes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
- L1: value 100uH -> 33uH; footprint Inductor_SMD:L_12x12mm_H6mm -> Inductor_SMD:L_Abracon_ASPI-0630LR; LCSC (none) -> https://www.lcsc.com/product-detail/Power-Inductors_cjiang-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
Connections:
- net +12V: now also U5.1 (VIN)
- net +5V: now also U5.4 (FB)
- net GND: now also U5.3 (GND), U5.5 (~{ON}/OFF)
- net at D3.1 (K), L1.1: now also U5.2 (OUT)
- no-connect marks 4 -> 1

Commit message: ....
Parts:
- added D4: 10V, symbol Device:D_Zener
- added R17: 2.2K, Resistor_SMD:R_0805_2012Metric, symbol Device:R
Connections:
- net +12V: now also D4.1 (K)
- net GND: now also R17.2
- new net: D4.2 (A), R17.1
Changed lines of the file:
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@@
+    (stroke (width 0) (type default))
+  )
+  (wire (pts (xy 124.46 149.86) (xy 124.46 156.21))
     (stroke (width 0) (type default))
   )
@@
     (stroke (width 0) (type default))
   )
+  (wire (pts (xy 124.46 125.73) (xy 124.46 128.27))
+    (stroke (width 0) (type default))
+  )
   (wire (pts (xy 209.55 49.53) (xy 212.09 49.53))
     (stroke (width 0) (type default))
@@
     (stroke (width 0) (type default))
   )
+  (wire (pts (xy 124.46 135.89) (xy 124.46 142.24))
+    (stroke (width 0) (type default))
+  )
   (wire (pts (xy 142.24 25.4) (xy 151.13 25.4))
     (stroke (width 0) (type default))
@@
   (label "TXD" (at 85.09 57.15 0) (fields_autoplaced)
     (effects (font (size 1.27 1.27)) (justify left bottom))
+  )
+  (symbol (lib_id "Device:D_Zener") (at 124.46 132.08 270) (unit 1)
+    (in_bom yes) (on_board yes) (dnp no)
+    (property "Reference" "D4" (at 127 130.81 90)
+      (effects (font (size 1.27 1.27)) (justify left))
+    )
+    (property "Value" "10V" (at 127 133.35 90)
+      (effects (font (size 1.27 1.27)) (justify left))
+    )
+    (property "Footprint" "" (at 124.46 132.08 0)
+      (effects (font (size 1.27 1.27)) hide)
+    )
+    (property "Datasheet" "~" (at 124.46 132.08 0)
+      (effects (font (size 1.27 1.27)) hide)
+    )
+    (property "part" "PDZ10B" (at 130.81 135.89 90)
+      (effects (font (size 1.27 1.27)))
+    )
+    (pin "1")
+    (pin "2")
+    (instances
+      (project "MasterShield"
+        (path "/16d5516d-cfb1-48ac-a57f-0957fae4baa5"
+          (reference "D4") (unit 1)
+        )
+      )
+    )
   )
   (symbol (lib_id "Connector:TestPoint") (at 92.71 57.15 180) (unit 1)
@@
         (path "/16d5516d-cfb1-48ac-a57f-0957fae4baa5"
           (reference "R4") (unit 1)
+        )
+      )
+    )
+  )
+  (symbol (lib_id "power:+12V") (at 124.46 125.73 0) (unit 1)
+    (in_bom yes) (on_board yes) (dnp no) (fields_autoplaced)
+    (property "Reference" "#PWR018" (at 124.46 129.54 0)
+      (effects (font (size 1.27 1.27)) hide)
+    )
+    (property "Value" "+12V" (at 124.46 120.65 0)
+      (effects (font (size 1.27 1.27)))
+    )
+    (property "Footprint" "" (at 124.46 125.73 0)
+      (effects (font (size 1.27 1.27)) hide)
+    )
+    (property "Datasheet" "" (at 124.46 125.73 0)
+      (effects (font (size 1.27 1.27)) hide)
+    )
+    (pin "1")
+    (instances
+      (project "MasterShield"
+        (path "/16d5516d-cfb1-48ac-a57f-0957fae4baa5"
+          (reference "#PWR018") (unit 1)
         )
       )
@@
     )
   )
+  (symbol (lib_id "power:GND") (at 124.46 156.21 0) (unit 1)
+    (in_bom yes) (on_board yes) (dnp no)
+    (property "Reference" "#PWR019" (at 124.46 162.56 0)
+      (effects (font (size 1.27 1.27)) hide)
+    )
+    (property "Value" "GND" (at 124.46 160.02 0)
+      (effects (font (size 1.27 1.27)))
+    )
+    (property "Footprint" "" (at 124.46 156.21 0)
+      (effects (font (size 1.27 1.27)) hide)
+    )
+    (property "Datasheet" "" (at 124.46 156.21 0)
+      (effects (font (size 1.27 1.27)) hide)
+    )
+    (pin "1")
+    (instances
+      (project "MasterShield"
+        (path "/16d5516d-cfb1-48ac-a57f-0957fae4baa5"
+          (reference "#PWR019") (unit 1)
+        )
+      )
+    )
+  )
   (symbol (lib_id "power:+5V") (at 95.25 93.98 90) (unit 1)
     (in_bom yes) (on_board yes) (dnp no) (fields_autoplaced)
@@
         )
       )
+    )
+  )
+  (symbol (lib_id "Device:R") (at 124.46 146.05 0) (unit 1)
+    (in_bom yes) (on_board yes) (dnp no) (fields_autoplaced)
+    (property "Reference" "R17" (at 127 144.78 0)
+      (effects (font (size 1.27 1.27)) (justify left))
+    )
+    (property "Value" "2.2K" (at 127 147.32 0)
+      (effects (font (size 1.27 1.27)) (justify left))
+    )
+    (property "Footprint" "Resistor_SMD:R_0805_2012Metric" (at 122.682 146.05 90)
+      (effects (font (size 1.27 1.27)) hide)
+    )
+    (property "Datasheet" "~" (at 124.46 146.05 0)
+      (effects (font (size 1.27 1.27)) hide)
+    )
+    (pin "1")
+    (pin "2")
+    (instances
+      (project "MasterShield"
+        (path "/16d5516d-cfb1-48ac-a57f-0957fae4baa5"
+          (reference "R17") (unit 1)
+        )
+      )

Commit message: ...
Parts:
- added D5: SS53C, Diode_SMD:D_SOD-323_HandSoldering, symbol Diode:1N5817
- added R20: 4.7K, Resistor_SMD:R_0805_2012Metric, symbol Device:R
- added R21: 10K, Resistor_SMD:R_0805_2012Metric, symbol Device:R
- added U4: LM321, Package_TO_SOT_SMD:SOT-23-5, symbol Amplifier_Operational:LM321
- D4: footprint (none) -> Diode_SMD:D_SOD-323_HandSoldering
- R17: value 2.2K -> 4.7k
Connections:
- net +3.3V: now also D5.1 (K)
- net +5V: now also U4.5 (V+)
- net AD0: now also D5.2 (A), R20.1, R21.1
- net GND: now also R21.2, U4.2 (V-)
- net at D4.2 (A), R17.1: now also U4.1 (+)
- new net: R20.2, U4.3 (-), U4.4
Other:
- note added: "Battery fuel gauge"
- note added: "Power load switch"
- note added: "UART to RS-485 converter"
- note added: "Voltage regulator"
- moved on the sheet: C4, C5, D3, D4, J6, L1, R12, R13, R17, U2, U5

Commit message: ...
Changed lines of the file:
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@@
     (stroke (width 0) (type default))
   )
-  (wire (pts (xy 25.4 85.09) (xy 34.29 85.09))
+  (wire (pts (xy 25.4 85.09) (xy 53.34 85.09))
     (stroke (width 0) (type default))
   )
@@
   )
   (label "AD0" (at 30.48 85.09 0) (fields_autoplaced)
+    (effects (font (size 1.27 1.27)) (justify left bottom))
+  )
+  (label "FUEL_GAUGE" (at 41.91 85.09 0) (fields_autoplaced)
     (effects (font (size 1.27 1.27)) (justify left bottom))
   )
@@
     (effects (font (size 1.27 1.27)) (justify left bottom))
   )
-  (label "AD0" (at 153.67 160.02 0) (fields_autoplaced)
-    (effects (font (size 1.27 1.27)) (justify left bottom))
-  )
   (label "RXD" (at 85.09 49.53 0) (fields_autoplaced)
     (effects (font (size 1.27 1.27)) (justify left bottom))
@@
     (effects (font (size 1.27 1.27)) (justify left bottom))
   )
+  (label "FUEL_GAUGE" (at 147.32 160.02 0) (fields_autoplaced)
+    (effects (font (size 1.27 1.27)) (justify left bottom))
+  )

Commit message: Added OV/UV/RP protection
Parts:
- added D6: LED, LED_SMD:LED_0805_2012Metric, symbol Device:LED
- added Q2: Si9945AEY-T1, Package_SO:SOP-8_3.9x4.9mm_P1.27mm, symbol Device:Q_Dual_NMOS_S1G1S2G2D2D2D1D1
- added Q3: S8050, Package_TO_SOT_SMD:SOT-23, symbol Transistor_BJT:S8050
- added R18: 2700k, Resistor_SMD:R_0805_2012Metric, symbol Device:R
- added R19, R22: 82k, Resistor_SMD:R_0805_2012Metric, symbol Device:R
- added R23, R25: 100k, Resistor_SMD:R_0805_2012Metric, symbol Device:R
- added R24: 1K, Resistor_SMD:R_0805_2012Metric, symbol Device:R
- added R26: 4.7K, Resistor_SMD:R_0805_2012Metric, symbol Device:R
- added U6: LTC4365TS8, Package_TO_SOT_SMD:TSOT-23-8, symbol Power_Management:LTC4365TS8
Connections:
- net +12V: now also Q2.5 (D), Q2.6 (D), U6.7 (Vout)
- net AD4: now also R13.2, U2.4 (ST1/2)
- net AD5: now also R12.2, U2.8 (ST3/4)
- net GND: now also Q3.1 (E), R22.2, R25.2, U6.4 (GND)
- net P0.08: now also R26.2; no longer R13.2, U2.4 (ST1/2)
- net P0.09: no longer R12.2, U2.8 (ST3/4)
- new net: R18.2, R19.1, U6.2 (UV)
- new net: R19.2, R22.1, U6.3 (OV)
- new net: D6.1 (K), U6.6 (~{FAULT})
- new net: D6.2 (A), R24.2
- new net: Q3.3 (C), R23.2, U6.5 (~{SHDN})
- new net: Q3.2 (B), R25.1, R26.1
- new net: Q2.1 (S), Q2.3 (S)
- new net: Q2.2 (G), Q2.4 (G), U6.8 (GATE)
- new net +BATT: Q2.7 (D), Q2.8 (D), R18.1, R23.1, R24.1, U6.1 (Vin)
Other:
- note added: "Power input protection"
- moved on the sheet: C4, C5, D3, D4, D5, L1, R17, R20, R21, U4, U5

Commit message: ...
Parts:
- added J7: BATT, TerminalBlock_4Ucon:TerminalBlock_4Ucon_1x04_P3.50mm_Horizontal, symbol Connector:Screw_Terminal_01x04
- added TP10: FUGA, TestPoint:TestPoint_Pad_D2.0mm, symbol Connector:TestPoint
- added TP11: POWER_EN4, TestPoint:TestPoint_Pad_D2.0mm, symbol Connector:TestPoint
- added TP12: POWER_EN3, TestPoint:TestPoint_Pad_D2.0mm, symbol Connector:TestPoint
- added TP13: POWER_EN2, TestPoint:TestPoint_Pad_D2.0mm, symbol Connector:TestPoint
- added TP14: POWER_EN1, TestPoint:TestPoint_Pad_D2.0mm, symbol Connector:TestPoint
- added TP15: POWER_ST12, TestPoint:TestPoint_Pad_D2.0mm, symbol Connector:TestPoint
- added TP16: POWER_ST34, TestPoint:TestPoint_Pad_D2.0mm, symbol Connector:TestPoint
- added TP17: GATE, TestPoint:TestPoint_Pad_D2.0mm, symbol Connector:TestPoint
- added TP5: UV, TestPoint:TestPoint_Pad_D2.0mm, symbol Connector:TestPoint
- added TP6: OV, TestPoint:TestPoint_Pad_D2.0mm, symbol Connector:TestPoint
- added TP7: SHDN, TestPoint:TestPoint_Pad_D2.0mm, symbol Connector:TestPoint
- added TP8: FAULT, TestPoint:TestPoint_Pad_D2.0mm, symbol Connector:TestPoint
- added TP9: FUEL_GAUGE, TestPoint:TestPoint_Pad_D2.0mm, symbol Connector:TestPoint
Connections:
- net +BATT: now also J7.3 (Pin_3), J7.4 (Pin_4)
- net AD0: now also TP9.1
- net AD4: now also TP15.1
- net AD5: now also TP16.1
- net GND: now also J7.1 (Pin_1), J7.2 (Pin_2)
- net P0.04: now also TP14.1
- net P0.05: now also TP13.1
- net P0.06: now also TP12.1
- net P0.07: now also TP11.1
- net P0.08: now also TP7.1
- net at D4.2 (A), R17.1, U4.1 (+): now also TP10.1
- net at R18.2, R19.1, U6.2 (UV): now also TP5.1
- net at R19.2, R22.1, U6.3 (OV): now also TP6.1
- net at D6.1 (K), U6.6 (~{FAULT}): now also TP8.1
- net at Q2.2 (G), Q2.4 (G), U6.8 (GATE): now also TP17.1
