File: MasterShield.kicad_sch (KiCad schematic)
At the start: 71 parts, among them J1 Conn_01x08_Pin, J2 Conn_01x10_Pin, J3 Conn_01x06_Pin, J4 Conn_01x08_Pin, J5 RS485, J6 Screw_Terminal_01x08, J7 BATT, Q1 S8050, Q2 Si9945AEY-T1, Q3 S8050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

Commit message: ...
Parts:
- C5: LCSC https://www.lcsc.com/product-detail/Tantalum-Capacitors_KEM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 -> (none); lcsc (none) -> https://www.lcsc.com/product-detail/Tantalum-Capacitors_KEM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
- D1, D2: color (none) -> green; lcsc (none) -> https://www.lcsc.com/product-detail/Light-Emitting-Diodes-L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; mouser (none) -> https://eu.mouser.com/ProductDetail/Broadcom-Avago/HSMM-C17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
- D3, D5: LCSCL https://www.lcsc.com/product-detail/Schottky-Barrier-Diodes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 -> (none); lcsc (none) -> https://www.lcsc.com/product-detail/Schottky-Barrier-Diodes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; mouser (none) -> https://eu.mouser.com/ProductDetail/Taiwan-Semiconductor/SK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
- D4: lcsc (none) -> https://www.lcsc.com/product-detail/Zener-Diodes_Nexperia-P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; mouser (none) -> https://eu.mouser.com/ProductDetail/Nexperia/PDZ10B115?qs=L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
- D6: color (none) -> red; lcsc (none) -> https://www.lcsc.com/product-detail/Light-Emitting-Diodes-s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; mouser (none) -> https://eu.mouser.com/ProductDetail/Broadcom-Avago/HSMH-H17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
- L1: LCSC https://www.lcsc.com/product-detail/Power-Inductors_cjiang-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 -> (none); lcsc (none) -> https://www.lcsc.com/product-detail/Power-Inductors_cjiang-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
- Q1, Q3: lcsc (none) -> https://www.lcsc.com/product-detail/Bipolar-Transistors-BJT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; mouser (none) -> https://eu.mouser.com/ProductDetail/Comchip-Technology/SS80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
- Q2: mouser (none) -> https://eu.mouser.com/ProductDetail/Vishay-Semiconductors/S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
- U1: lcsc (none) -> https://www.lcsc.com/product-detail/RS-span-style-backgroun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; mouser (none) -> https://eu.mouser.com/ProductDetail/Analog-Devices-Maxim-In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
- U2: lcsc (none) -> https://www.lcsc.com/product-detail/Power-Distribution-Swit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; mouser (none) -> https://eu.mouser.com/ProductDetail/Infineon-Technologies/B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
- U3: lcsc (none) -> https://www.lcsc.com/product-detail/Gates_Nexperia-74LVC1G0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; mouser (none) -> https://eu.mouser.com/ProductDetail/Nexperia/74LVC1G08GW-Q1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
- U4: lcsc (none) -> https://www.lcsc.com/product-detail/Operational-Amplifier_X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; mouser (none) -> https://eu.mouser.com/ProductDetail/Texas-Instruments/LM321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
- U5: LCSC https://www.lcsc.com/product-detail/DC-DC-Converters_Texas-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 -> (none); lcsc (none) -> https://www.lcsc.com/product-detail/DC-DC-Converters_Texas-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; mouser (none) -> https://eu.mouser.com/ProductDetail/Texas-Instruments/LM259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
- U6: mouser (none) -> https://eu.mouser.com/ProductDetail/Analog-Devices/LTC4365H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
Changed lines of the file:
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@@
       (effects (font (size 1.27 1.27)))
+    )
+    (property "lcsc" "https://www.lcsc.com/product-detail/Zener-Diodes_Nexperia-PDZ10B-115_C85383.html" (at 73.66 147.32 90)
+      (effects (font (size 1.27 1.27)) hide)
+    )
+    (property "mouser" "https://eu.mouser.com/ProductDetail/Nexperia/PDZ10B115?qs=LOCUfHb8d9t6BsAtogB8tA%3D%3D" (at 73.66 147.32 90)
+      (effects (font (size 1.27 1.27)) hide)
     )
     (pin "1")
@@
       (effects (font (size 1.27 1.27)) hide)
     )
+    (property "lcsc" "https://www.lcsc.com/product-detail/Light-Emitting-Diodes-span-style-background-color-ff0-LED-span_Yongyu-Photoelectric-SZYY0805R_C434431.html" (at 139.7 124.46 90)
+      (effects (font (size 1.27 1.27)) hide)
+    )
+    (property "mouser" "https://eu.mouser.com/ProductDetail/Broadcom-Avago/HSMH-H170?qs=Li%252BoUPsLEns3UdNxsKqV%252Bg%3D%3D" (at 139.7 124.46 90)
+      (effects (font (size 1.27 1.27)) hide)
+    )
+    (property "color" "red" (at 142.24 124.46 0)
+      (effects (font (size 1.27 1.27)))
+    )
     (pin "1")
     (pin "2")
@@
       (effects (font (size 1.27 1.27)) hide)
     )
-    (property "LCSCL" "https://www.lcsc.com/product-detail/Schottky-Barrier-Diodes-SBD_LGE-SS53C_C330397.html" (at 246.38 110.49 90)
+    (property "lcsc" "https://www.lcsc.com/product-detail/Schottky-Barrier-Diodes-SBD_LGE-SS53C_C330397.html" (at 246.38 110.49 90)
+      (effects (font (size 1.27 1.27)) hide)
+    )
+    (property "mouser" "https://eu.mouser.com/ProductDetail/Taiwan-Semiconductor/SK53C?qs=tHU%2FlV7kTyQZH0fUzmR2AA%3D%3D" (at 246.38 110.49 90)
       (effects (font (size 1.27 1.27)) hide)
     )
@@
   )
   (symbol (lib_id "Device:LED") (at 88.9 30.48 90) (unit 1)
-    (in_bom yes) (on_board yes) (dnp no) (fields_autoplaced)
+    (in_bom yes) (on_board yes) (dnp no)
     (property "Reference" "D2" (at 92.71 30.7975 90)
       (effects (font (size 1.27 1.27)) (justify right))
@@
     (property "Datasheet" "~" (at 88.9 30.48 0)
       (effects (font (size 1.27 1.27)) hide)
+    )
+    (property "lcsc" "https://www.lcsc.com/product-detail/Light-Emitting-Diodes-LED_Foshan-NationStar-Optoelectronics-NCD0805C1_C84257.html" (at 88.9 30.48 90)
+      (effects (font (size 1.27 1.27)) hide)
+    )
+    (property "mouser" "https://eu.mouser.com/ProductDetail/Broadcom-Avago/HSMM-C170?qs=YDL0qNrpDT515hwcVWI5gg%3D%3D" (at 88.9 30.48 90)
+      (effects (font (size 1.27 1.27)) hide)
+    )
+    (property "color" "green" (at 91.44 29.21 0)
+      (effects (font (size 1.27 1.27)))
     )
     (pin "1")
@@
     (property "Datasheet" "http://www.unisonic.com.tw/datasheet/S8050.pdf" (at 167.64 132.08 0)
       (effects (font (size 1.27 1.27)) (justify left) hide)
+    )
+    (property "lcsc" "https://www.lcsc.com/product-detail/Bipolar-Transistors-BJT_JSMSEMI-S8050_C916390.html" (at 167.64 132.08 0)
+      (effects (font (size 1.27 1.27)) hide)
+    )
+    (property "mouser" "https://eu.mouser.com/ProductDetail/Comchip-Technology/SS8050-G?qs=LLUE9lz1YbcHg%252BWLMAtcrQ%3D%3D" (at 167.64 132.08 0)
+      (effects (font (size 1.27 1.27)) hide)
     )
     (pin "1")
@@
       (effects (font (size 1.27 1.27)) hide)
     )
+    (property "lcsc" "https://www.lcsc.com/product-detail/Gates_Nexperia-74LVC1G08GW-125_C12512.html" (at 109.22 93.98 90)
+      (effects (font (size 1.27 1.27)) hide)
+    )
+    (property "mouser" "https://eu.mouser.com/ProductDetail/Nexperia/74LVC1G08GW-Q1001?qs=1sbE9T7hb3YW60vUdTya5Q%3D%3D" (at 109.22 93.98 90)
+      (effects (font (size 1.27 1.27)) hide)
+    )
     (pin "1")
     (pin "2")
@@
       (effects (font (size 1.27 1.27)) hide)
     )
-    (property "LCSC" "https://www.lcsc.com/product-detail/Power-Inductors_cjiang-Changjiang-Microelectronics-Tech-FXL0630-330-M_C177245.html" (at 256.54 104.14 90)
+    (property "lcsc" "https://www.lcsc.com/product-detail/Power-Inductors_cjiang-Changjiang-Microelectronics-Tech-FXL0630-330-M_C177245.html" (at 256.54 104.14 90)
       (effects (font (size 1.27 1.27)) hide)
     )
@@
     )
     (property "Datasheet" "https://www.infineon.com/dgdl/Infineon-BTS724G-DS-v01_00-EN.pdf?fileId=5546d4625a888733015aa3a2f1030ff1" (at 225.425 55.88 0)
+      (effects (font (size 1.27 1.27)) hide)
+    )
+    (property "lcsc" "https://www.lcsc.com/product-detail/Power-Distribution-Switches_Infineon-Technologies-BTS724G_C82656.html" (at 227.33 58.42 0)
+      (effects (font (size 1.27 1.27)) hide)
+    )
+    (property "mouser" "https://eu.mouser.com/ProductDetail/Infineon-Technologies/BTS724G?qs=MGskQgfwDzvkc3kAjdyGig%3D%3D" (at 227.33 58.42 0)
       (effects (font (size 1.27 1.27)) hide)
     )
@@
       (effects (font (size 1.27 1.27)) hide)
     )
+    (property "mouser" "https://eu.mouser.com/ProductDetail/Vishay-Semiconductors/SI9945BDY-T1-GE3?qs=%252BPu8jn5UVnFSRz4ameiu9g%3D%3D" (at 179.07 101.6 90)
+      (effects (font (size 1.27 1.27)) hide)
+    )
     (pin "1")
     (pin "2")
@@
       (effects (font (size 1.27 1.27)) hide)
     )
+    (property "lcsc" "https://www.lcsc.com/product-detail/RS-span-style-background-color-ff0-485-span-RS-422-ICs_HTC-Korea-TAEJIN-Tech-MAX485ED_C481667.html" (at 127 52.07 0)
+      (effects (font (size 1.27 1.27)) hide)
+    )
+    (property "mouser" "https://eu.mouser.com/ProductDetail/Analog-Devices-Maxim-Integrated/MAX485ESA%2bT?qs=LHmEVA8xxfYXmvxEk%252BFtEg%3D%3D" (at 127 52.07 0)
+      (effects (font (size 1.27 1.27)) hide)
+    )
     (pin "1")
     (pin "2")
@@
       (effects (font (size 1.27 1.27)) hide)
     )
+    (property "mouser" "https://eu.mouser.com/ProductDetail/Vishay-Semiconductors/SI9945BDY-T1-GE3?qs=%252BPu8jn5UVnFSRz4ameiu9g%3D%3D" (at 189.23 101.6 90)
+      (effects (font (size 1.27 1.27)) hide)
+    )
     (pin "1")
     (pin "2")
@@
   )
   (symbol (lib_id "Device:LED") (at 99.06 30.48 90) (unit 1)
-    (in_bom yes) (on_board yes) (dnp no) (fields_autoplaced)
+    (in_bom yes) (on_board yes) (dnp no)
     (property "Reference" "D1" (at 102.87 30.7975 90)
       (effects (font (size 1.27 1.27)) (justify right))
@@
       (effects (font (size 1.27 1.27)) hide)
     )
+    (property "lcsc" "https://www.lcsc.com/product-detail/Light-Emitting-Diodes-LED_Foshan-NationStar-Optoelectronics-NCD0805C1_C84257.html" (at 99.06 30.48 90)
+      (effects (font (size 1.27 1.27)) hide)
+    )
+    (property "mouser" "https://eu.mouser.com/ProductDetail/Broadcom-Avago/HSMM-C170?qs=YDL0qNrpDT515hwcVWI5gg%3D%3D" (at 99.06 30.48 90)
+      (effects (font (size 1.27 1.27)) hide)
+    )
+    (property "color" "green" (at 101.6 29.21 0)
+      (effects (font (size 1.27 1.27)))
+    )
     (pin "1")
     (pin "2")
@@
     )
     (property "lcsc" "https://www.lcsc.com/product-detail/Surge-Suppressors_Analog-Devices-LTC4365ITS8-TRPBF_C514441.html" (at 184.15 120.65 0)
+      (effects (font (size 1.27 1.27)) hide)
+    )
+    (property "mouser" "https://eu.mouser.com/ProductDetail/Analog-Devices/LTC4365HTS8WTRPBF?qs=BJlw7L4Cy7%252BIvjFg8vMT2w%3D%3D" (at 184.15 120.65 0)
       (effects (font (size 1.27 1.27)) hide)
     )
@@
     )
     (property "Datasheet" "http://www.ti.com/lit/ds/symlink/lm321.pdf" (at 95.25 157.48 0)
+      (effects (font (size 1.27 1.27)) hide)
+    )
+    (property "lcsc" "https://www.lcsc.com/product-detail/Operational-Amplifier_XBLW-LM321DTR-XBLW_C18723612.html" (at 95.25 157.48 0)
+      (effects (font (size 1.27 1.27)) hide)
+    )
+    (property "mouser" "https://eu.mouser.com/ProductDetail/Texas-Instruments/LM321MF-NOPB?qs=X1J7HmVL2ZEjaSKPrGsivQ%3D%3D" (at 95.25 157.48 0)
       (effects (font (size 1.27 1.27)) hide)
     )
@@
       (effects (font (size 1.27 1.27)) hide)
     )
-    (property "LCSC" "https://www.lcsc.com/product-detail/DC-DC-Converters_Texas-Instruments-LM2596SX-5-0-NOPB_C10002.html" (at 233.68 101.6 0)
+    (property "lcsc" "https://www.lcsc.com/product-detail/DC-DC-Converters_Texas-Instruments-LM2596SX-5-0-NOPB_C10002.html" (at 233.68 101.6 0)
+      (effects (font (size 1.27 1.27)) hide)
+    )
+    (property "mouser" "https://eu.mouser.com/ProductDetail/Texas-Instruments/LM2596S-5.0-NOPB?qs=X1J7HmVL2ZHVjCOmW%252BYINA%3D%3D" (at 233.68 101.6 0)
       (effects (font (size 1.27 1.27)) hide)
     )
@@
       (effects (font (size 1.27 1.27)) (justify left) hide)
     )
+    (property "lcsc" "https://www.lcsc.com/product-detail/Bipolar-Transistors-BJT_JSMSEMI-S8050_C916390.html" (at 96.52 69.85 0)
+      (effects (font (size 1.27 1.27)) hide)
+    )
+    (property "mouser" "https://eu.mouser.com/ProductDetail/Comchip-Technology/SS8050-G?qs=LLUE9lz1YbcHg%252BWLMAtcrQ%3D%3D" (at 96.52 69.85 0)
+      (effects (font (size 1.27 1.27)) hide)
+    )
     (pin "1")
     (pin "2")
@@
       (effects (font (size 1.27 1.27)) hide)
     )
-    (property "LCSCL" "https://www.lcsc.com/product-detail/Schottky-Barrier-Diodes-SBD_LGE-SS53C_C330397.html" (at 125.73 148.59 90)
+    (property "lcsc" "https://www.lcsc.com/product-detail/Schottky-Barrier-Diodes-SBD_LGE-SS53C_C330397.html" (at 125.73 148.59 90)
+      (effects (font (size 1.27 1.27)) hide)
+    )
+    (property "mouser" "https://eu.mouser.com/ProductDetail/Taiwan-Semiconductor/SK53C?qs=tHU%2FlV7kTyQZH0fUzmR2AA%3D%3D" (at 125.73 148.59 90)
       (effects (font (size 1.27 1.27)) hide)
     )
@@
       (effects (font (size 1.27 1.27)) hide)
     )
-    (property "LCSC" "https://www.lcsc.com/product-detail/Tantalum-Capacitors_KEMET-T491D227K016AT_C122304.html" (at 267.97 111.76 0)
-      (effects (font (size 1.27 1.27)) hide)
-    )
+    (property "lcsc" "https://www.lcsc.com/product-detail/Tantalum-Capacitors_KEMET-T491D227K016AT_C122304.html" (at 267.97 111.76 0)
+      (effects (font (size 1.27 1.27)) hide)
+    )

Commit message: ...
Parts:
- J1: value Conn_01x08_Pin -> CONTROL/SERIAL
- J2: value Conn_01x10_Pin -> MISC
- J3: value Conn_01x06_Pin -> ADC/SENSE
- J4: value Conn_01x08_Pin -> POWER
Changed lines of the file:
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@@
       (effects (font (size 1.27 1.27)))
     )
-    (property "Value" "Conn_01x06_Pin" (at 20.955 82.55 0)
+    (property "Value" "ADC/SENSE" (at 20.955 82.55 0)
       (effects (font (size 1.27 1.27)))
     )
@@
       (effects (font (size 1.27 1.27)))
     )
-    (property "Value" "Conn_01x08_Pin" (at 20.955 21.59 0)
+    (property "Value" "CONTROL/SERIAL" (at 20.955 21.59 0)
       (effects (font (size 1.27 1.27)))
     )
@@
       (effects (font (size 1.27 1.27)))
     )
-    (property "Value" "Conn_01x08_Pin" (at 20.955 105.41 0)
+    (property "Value" "POWER" (at 20.955 105.41 0)
       (effects (font (size 1.27 1.27)))
     )
@@
       (effects (font (size 1.27 1.27)))
     )
-    (property "Value" "Conn_01x10_Pin" (at 21.59 48.26 0)
-      (effects (font (size 1.27 1.27)))
-    )
+    (property "Value" "MISC" (at 21.59 48.26 0)
+      (effects (font (size 1.27 1.27)))
+    )

Commit message: ...
Parts:
- removed TP11: POWER_EN4, TestPoint:TestPoint_Pad_D2.0mm, symbol Connector:TestPoint
- removed TP12: POWER_EN3, TestPoint:TestPoint_Pad_D2.0mm, symbol Connector:TestPoint
- removed TP13: POWER_EN2, TestPoint:TestPoint_Pad_D2.0mm, symbol Connector:TestPoint
- removed TP14: POWER_EN1, TestPoint:TestPoint_Pad_D2.0mm, symbol Connector:TestPoint
- removed TP15: POWER_ST12, TestPoint:TestPoint_Pad_D2.0mm, symbol Connector:TestPoint
- removed TP16: POWER_ST34, TestPoint:TestPoint_Pad_D2.0mm, symbol Connector:TestPoint
- D1: value LED -> RXD
- D2: value LED -> TXD
Changed lines of the file:
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@@
-    )
-  )
-  (symbol (lib_id "Connector:TestPoint") (at 57.15 36.83 270) (unit 1)
-    (in_bom yes) (on_board yes) (dnp no)
-    (property "Reference" "TP13" (at 66.04 36.83 90)
-      (effects (font (size 1.27 1.27)) (justify right))
-    )
-    (property "Value" "POWER_EN2" (at 77.47 36.83 90)
-      (effects (font (size 1.27 1.27)) (justify right))
-    )
-    (property "Footprint" "TestPoint:TestPoint_Pad_D2.0mm" (at 57.15 41.91 0)
-      (effects (font (size 1.27 1.27)) hide)
-    )
-    (property "Datasheet" "~" (at 57.15 41.91 0)
-      (effects (font (size 1.27 1.27)) hide)
-    )
-    (pin "1")
-    (instances
-      (project "MasterShield"
-        (path "/16d5516d-cfb1-48ac-a57f-0957fae4baa5"
-          (reference "TP13") (unit 1)
-        )
-      )
     )
   )
@@
     )
   )
-  (symbol (lib_id "Connector:TestPoint") (at 57.15 95.25 270) (unit 1)
-    (in_bom yes) (on_board yes) (dnp no)
-    (property "Reference" "TP15" (at 67.31 95.25 90)
-      (effects (font (size 1.27 1.27)) (justify right))
-    )
-    (property "Value" "POWER_ST12" (at 80.01 95.25 90)
-      (effects (font (size 1.27 1.27)) (justify right))
-    )
-    (property "Footprint" "TestPoint:TestPoint_Pad_D2.0mm" (at 57.15 100.33 0)
-      (effects (font (size 1.27 1.27)) hide)
-    )
-    (property "Datasheet" "~" (at 57.15 100.33 0)
-      (effects (font (size 1.27 1.27)) hide)
-    )
-    (pin "1")
-    (instances
-      (project "MasterShield"
-        (path "/16d5516d-cfb1-48ac-a57f-0957fae4baa5"
-          (reference "TP15") (unit 1)
-        )
-      )
-    )
-  )
   (symbol (lib_id "power:+5V") (at 127 22.86 0) (unit 1)
     (in_bom yes) (on_board yes) (dnp no) (fields_autoplaced)
@@
       (effects (font (size 1.27 1.27)) (justify right))
     )
-    (property "Value" "LED" (at 92.71 33.3375 90)
+    (property "Value" "TXD" (at 92.71 33.3375 90)
       (effects (font (size 1.27 1.27)) (justify right))
     )
@@
     )
   )
-  (symbol (lib_id "Connector:TestPoint") (at 57.15 39.37 270) (unit 1)
-    (in_bom yes) (on_board yes) (dnp no)
-    (property "Reference" "TP12" (at 66.04 39.37 90)
-      (effects (font (size 1.27 1.27)) (justify right))
-    )
-    (property "Value" "POWER_EN3" (at 77.47 39.37 90)
-      (effects (font (size 1.27 1.27)) (justify right))
-    )
-    (property "Footprint" "TestPoint:TestPoint_Pad_D2.0mm" (at 57.15 44.45 0)
-      (effects (font (size 1.27 1.27)) hide)
-    )
-    (property "Datasheet" "~" (at 57.15 44.45 0)
-      (effects (font (size 1.27 1.27)) hide)
-    )
-    (pin "1")
-    (instances
-      (project "MasterShield"
-        (path "/16d5516d-cfb1-48ac-a57f-0957fae4baa5"
-          (reference "TP12") (unit 1)
-        )
-      )
-    )
-  )
   (symbol (lib_id "Device:R") (at 214.63 40.64 0) (unit 1)
     (in_bom yes) (on_board yes) (dnp no)
@@
       (effects (font (size 1.27 1.27)) (justify right))
     )
-    (property "Value" "LED" (at 102.87 33.3375 90)
+    (property "Value" "RXD" (at 102.87 33.3375 90)
       (effects (font (size 1.27 1.27)) (justify right))
     )
@@
         (path "/16d5516d-cfb1-48ac-a57f-0957fae4baa5"
           (reference "D1") (unit 1)
-        )
-      )
-    )
-  )
-  (symbol (lib_id "Connector:TestPoint") (at 57.15 41.91 270) (unit 1)
-    (in_bom yes) (on_board yes) (dnp no)
-    (property "Reference" "TP11" (at 66.04 41.91 90)
-      (effects (font (size 1.27 1.27)) (justify right))
-    )
-    (property "Value" "POWER_EN4" (at 77.47 41.91 90)
-      (effects (font (size 1.27 1.27)) (justify right))
-    )
-    (property "Footprint" "TestPoint:TestPoint_Pad_D2.0mm" (at 57.15 46.99 0)
-      (effects (font (size 1.27 1.27)) hide)
-    )
-    (property "Datasheet" "~" (at 57.15 46.99 0)
-      (effects (font (size 1.27 1.27)) hide)
-    )
-    (pin "1")
-    (instances
-      (project "MasterShield"
-        (path "/16d5516d-cfb1-48ac-a57f-0957fae4baa5"
-          (reference "TP11") (unit 1)
         )
       )
@@
     )
   )
-  (symbol (lib_id "Connector:TestPoint") (at 57.15 34.29 270) (unit 1)
-    (in_bom yes) (on_board yes) (dnp no)
-    (property "Reference" "TP14" (at 66.04 34.29 90)
-      (effects (font (size 1.27 1.27)) (justify right))
-    )
-    (property "Value" "POWER_EN1" (at 77.47 34.29 90)
-      (effects (font (size 1.27 1.27)) (justify right))
-    )
-    (property "Footprint" "TestPoint:TestPoint_Pad_D2.0mm" (at 57.15 39.37 0)
-      (effects (font (size 1.27 1.27)) hide)
-    )
-    (property "Datasheet" "~" (at 57.15 39.37 0)
-      (effects (font (size 1.27 1.27)) hide)
-    )
-    (pin "1")
-    (instances
-      (project "MasterShield"
-        (path "/16d5516d-cfb1-48ac-a57f-0957fae4baa5"
-          (reference "TP14") (unit 1)
-        )
-      )
-    )
-  )
   (symbol (lib_id "Device:R") (at 209.55 40.64 0) (unit 1)
     (in_bom yes) (on_board yes) (dnp no)
@@
         )
       )
-    )
-  )
-  (symbol (lib_id "Connector:TestPoint") (at 57.15 97.79 270) (unit 1)
-    (in_bom yes) (on_board yes) (dnp no)
-    (property "Reference" "TP16" (at 67.31 97.79 90)
-      (effects (font (size 1.27 1.27)) (justify right))
-    )
-    (property "Value" "POWER_ST34" (at 80.01 97.79 90)
-      (effects (font (size 1.27 1.27)) (justify right))
-    )
-    (property "Footprint" "TestPoint:TestPoint_Pad_D2.0mm" (at 57.15 102.87 0)
-      (effects (font (size 1.27 1.27)) hide)
-    )
-    (property "Datasheet" "~" (at 57.15 102.87 0)
-      (effects (font (size 1.27 1.27)) hide)
-    )
-    (pin "1")
-    (instances
-      (project "MasterShield"
-        (path "/16d5516d-cfb1-48ac-a57f-0957fae4baa5"
-          (reference "TP16") (unit 1)
-        )
-      )

Commit message: ...
Connections:
- net +5V: now also C3.1; no longer C3.2, J5.1 (Pin_1)
- net AD4: now also R12.2, U2.8 (ST3/4); no longer R13.2, U2.4 (ST1/2)
- net AD5: now also R13.2, U2.4 (ST1/2); no longer R12.2, U2.8 (ST3/4)
- net GND: now also C3.2; no longer C3.1
- net at J6.7 (Pin_7), U2.13 (OUT4): now also J5.1 (Pin_1)
Other:
- moved on the sheet: C2, C3

Commit message: ...
Parts:
- removed J6: Screw_Terminal_01x08, TerminalBlock_4Ucon:TerminalBlock_4Ucon_1x08_P3.50mm_Horizontal, symbol Connector:Screw_Terminal_01x08
- added J6: EXTRA POWER, TerminalBlock_4Ucon:TerminalBlock_4Ucon_1x04_P3.50mm_Horizontal, symbol Connector:Screw_Terminal_01x04
- added J8: RS485 A, TerminalBlock_4Ucon:TerminalBlock_4Ucon_1x04_P3.50mm_Horizontal, symbol Connector:Screw_Terminal_01x04
- J5: value RS485 -> RS485 B
- R6: value R120 -> 120R
- R7: value R10 -> 10R
Connections:
- net GND: now also J6.1 (Pin_1), J6.4 (Pin_4), J8.2 (Pin_2)
- net at U2.18 (OUT1): now also J6.2 (Pin_2)
- net at U2.17 (OUT2): now also J6.3 (Pin_3)
- net at U2.14 (OUT3): now also J5.1 (Pin_1)
- net at U2.13 (OUT4): now also J8.1 (Pin_1); no longer J5.1 (Pin_1)
- net at J5.3 (Pin_3), R6.2, R7.1: now also J8.3 (Pin_3)
- net at J5.4 (Pin_4), R5.2, R6.1: now also J8.4 (Pin_4)

Commit message: ...
Parts:
- J5: value RS485 B -> RS485 A
- J8: value RS485 A -> RS485 B
Changed lines of the file:
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@@
       (effects (font (size 1.27 1.27)) (justify left))
     )
-    (property "Value" "RS485 B" (at 170.18 43.18 0)
+    (property "Value" "RS485 A" (at 170.18 43.18 0)
       (effects (font (size 1.27 1.27)) (justify left))
     )
@@
       (effects (font (size 1.27 1.27)) (justify left))
     )
-    (property "Value" "RS485 A" (at 170.18 27.94 0)
-      (effects (font (size 1.27 1.27)) (justify left))
-    )
+    (property "Value" "RS485 B" (at 170.18 27.94 0)
+      (effects (font (size 1.27 1.27)) (justify left))
+    )
