File: MasterShield.kicad_sch (KiCad schematic)
At the start: 66 parts, among them J1 CONTROL/SERIAL, J2 MISC, J3 ADC/SENSE, J4 POWER, J5 RS485 A, J6 EXTRA POWER, J7 BATT, J8 RS485 B, Q1 S8050, Q2 Si9945AEY-T1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

Commit message: ...
Parts:
- C5: LCSC (none) -> https://www.lcsc.com/product-detail/Tantalum-Capacitors_KEM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; lcsc https://www.lcsc.com/product-detail/Tantalum-Capacitors_KEM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 -> (none)
- D1, D2: LCSC (none) -> https://www.lcsc.com/product-detail/Light-Emitting-Diodes-L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; lcsc https://www.lcsc.com/product-detail/Light-Emitting-Diodes-L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 -> (none)
- D3, D5: LCSC (none) -> https://www.lcsc.com/product-detail/Schottky-Barrier-Diodes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; lcsc https://www.lcsc.com/product-detail/Schottky-Barrier-Diodes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 -> (none)
- D4: LCSC (none) -> https://www.lcsc.com/product-detail/Zener-Diodes_Nexperia-P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; lcsc https://www.lcsc.com/product-detail/Zener-Diodes_Nexperia-P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 -> (none)
- D6: LCSC (none) -> https://www.lcsc.com/product-detail/Light-Emitting-Diodes-s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; lcsc https://www.lcsc.com/product-detail/Light-Emitting-Diodes-s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 -> (none)
- L1: LCSC (none) -> https://www.lcsc.com/product-detail/Power-Inductors_cjiang-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; lcsc https://www.lcsc.com/product-detail/Power-Inductors_cjiang-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 -> (none)
- Q1, Q3: LCSC (none) -> https://www.lcsc.com/product-detail/Bipolar-Transistors-BJT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; lcsc https://www.lcsc.com/product-detail/Bipolar-Transistors-BJT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 -> (none)
- Q2: LCSC (none) -> https://www.lcsc.com/product-detail/MOSFETs_TECH-PUBLIC-SI9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; lcsc https://www.lcsc.com/product-detail/MOSFETs_TECH-PUBLIC-SI9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 -> (none)
- U1: LCSC (none) -> https://www.lcsc.com/product-detail/RS-span-style-backgroun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; lcsc https://www.lcsc.com/product-detail/RS-span-style-backgroun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 -> (none)
- U2: LCSC (none) -> https://www.lcsc.com/product-detail/Power-Distribution-Swit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; lcsc https://www.lcsc.com/product-detail/Power-Distribution-Swit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 -> (none)
- U3: LCSC (none) -> https://www.lcsc.com/product-detail/Gates_Nexperia-74LVC1G0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; lcsc https://www.lcsc.com/product-detail/Gates_Nexperia-74LVC1G0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 -> (none)
- U4: LCSC (none) -> https://www.lcsc.com/product-detail/Operational-Amplifier_X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; lcsc https://www.lcsc.com/product-detail/Operational-Amplifier_X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 -> (none)
- U5: LCSC (none) -> https://www.lcsc.com/product-detail/DC-DC-Converters_Texas-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; lcsc https://www.lcsc.com/product-detail/DC-DC-Converters_Texas-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 -> (none)
- U6: LCSC (none) -> https://www.lcsc.com/product-detail/Surge-Suppressors_Analo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; lcsc https://www.lcsc.com/product-detail/Surge-Suppressors_Analo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 -> (none)
Changed lines of the file:
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@@
       (effects (font (size 1.27 1.27)))
     )
-    (property "lcsc" "https://www.lcsc.com/product-detail/Zener-Diodes_Nexperia-PDZ10B-115_C85383.html" (at 73.66 147.32 90)
+    (property "LCSC" "https://www.lcsc.com/product-detail/Zener-Diodes_Nexperia-PDZ10B-115_C85383.html" (at 73.66 147.32 90)
       (effects (font (size 1.27 1.27)) hide)
     )
@@
       (effects (font (size 1.27 1.27)) hide)
     )
-    (property "lcsc" "https://www.lcsc.com/product-detail/Light-Emitting-Diodes-span-style-background-color-ff0-LED-span_Yongyu-Photoelectric-SZYY0805R_C434431.html" (at 139.7 124.46 90)
+    (property "LCSC" "https://www.lcsc.com/product-detail/Light-Emitting-Diodes-span-style-background-color-ff0-LED-span_Yongyu-Photoelectric-SZYY0805R_C434431.html" (at 139.7 124.46 90)
       (effects (font (size 1.27 1.27)) hide)
     )
@@
       (effects (font (size 1.27 1.27)) hide)
     )
-    (property "lcsc" "https://www.lcsc.com/product-detail/Schottky-Barrier-Diodes-SBD_LGE-SS53C_C330397.html" (at 246.38 110.49 90)
+    (property "LCSC" "https://www.lcsc.com/product-detail/Schottky-Barrier-Diodes-SBD_LGE-SS53C_C330397.html" (at 246.38 110.49 90)
       (effects (font (size 1.27 1.27)) hide)
     )
@@
       (effects (font (size 1.27 1.27)) hide)
     )
-    (property "lcsc" "https://www.lcsc.com/product-detail/Light-Emitting-Diodes-LED_Foshan-NationStar-Optoelectronics-NCD0805C1_C84257.html" (at 88.9 30.48 90)
+    (property "LCSC" "https://www.lcsc.com/product-detail/Light-Emitting-Diodes-LED_Foshan-NationStar-Optoelectronics-NCD0805C1_C84257.html" (at 88.9 30.48 90)
       (effects (font (size 1.27 1.27)) hide)
     )
@@
       (effects (font (size 1.27 1.27)) (justify left) hide)
     )
-    (property "lcsc" "https://www.lcsc.com/product-detail/Bipolar-Transistors-BJT_JSMSEMI-S8050_C916390.html" (at 167.64 132.08 0)
+    (property "LCSC" "https://www.lcsc.com/product-detail/Bipolar-Transistors-BJT_JSMSEMI-S8050_C916390.html" (at 167.64 132.08 0)
       (effects (font (size 1.27 1.27)) hide)
     )
@@
       (effects (font (size 1.27 1.27)) hide)
     )
-    (property "lcsc" "https://www.lcsc.com/product-detail/Gates_Nexperia-74LVC1G08GW-125_C12512.html" (at 109.22 93.98 90)
+    (property "LCSC" "https://www.lcsc.com/product-detail/Gates_Nexperia-74LVC1G08GW-125_C12512.html" (at 109.22 93.98 90)
       (effects (font (size 1.27 1.27)) hide)
     )
@@
       (effects (font (size 1.27 1.27)) hide)
     )
-    (property "lcsc" "https://www.lcsc.com/product-detail/Power-Inductors_cjiang-Changjiang-Microelectronics-Tech-FXL0630-330-M_C177245.html" (at 256.54 104.14 90)
+    (property "LCSC" "https://www.lcsc.com/product-detail/Power-Inductors_cjiang-Changjiang-Microelectronics-Tech-FXL0630-330-M_C177245.html" (at 256.54 104.14 90)
       (effects (font (size 1.27 1.27)) hide)
     )
@@
       (effects (font (size 1.27 1.27)) hide)
     )
-    (property "lcsc" "https://www.lcsc.com/product-detail/Power-Distribution-Switches_Infineon-Technologies-BTS724G_C82656.html" (at 227.33 58.42 0)
+    (property "LCSC" "https://www.lcsc.com/product-detail/Power-Distribution-Switches_Infineon-Technologies-BTS724G_C82656.html" (at 227.33 58.42 0)
       (effects (font (size 1.27 1.27)) hide)
     )
@@
       (effects (font (size 1.27 1.27)) hide)
     )
-    (property "lcsc" "https://www.lcsc.com/product-detail/MOSFETs_TECH-PUBLIC-SI9945AEY_C3040623.html" (at 179.07 101.6 90)
+    (property "LCSC" "https://www.lcsc.com/product-detail/MOSFETs_TECH-PUBLIC-SI9945AEY_C3040623.html" (at 179.07 101.6 90)
       (effects (font (size 1.27 1.27)) hide)
     )
@@
       (effects (font (size 1.27 1.27)) hide)
     )
-    (property "lcsc" "https://www.lcsc.com/product-detail/RS-span-style-background-color-ff0-485-span-RS-422-ICs_HTC-Korea-TAEJIN-Tech-MAX485ED_C481667.html" (at 127 52.07 0)
+    (property "LCSC" "https://www.lcsc.com/product-detail/RS-span-style-background-color-ff0-485-span-RS-422-ICs_HTC-Korea-TAEJIN-Tech-MAX485ED_C481667.html" (at 127 52.07 0)
       (effects (font (size 1.27 1.27)) hide)
     )
@@
       (effects (font (size 1.27 1.27)) hide)
     )
-    (property "lcsc" "https://www.lcsc.com/product-detail/MOSFETs_TECH-PUBLIC-SI9945AEY_C3040623.html" (at 189.23 101.6 90)
-      (effects (font (size 1.27 1.27)) hide)
-    )
     (property "mouser" "https://eu.mouser.com/ProductDetail/Vishay-Semiconductors/SI9945BDY-T1-GE3?qs=%252BPu8jn5UVnFSRz4ameiu9g%3D%3D" (at 189.23 101.6 90)
+      (effects (font (size 1.27 1.27)) hide)
+    )
+    (property "LCSC" "https://www.lcsc.com/product-detail/MOSFETs_TECH-PUBLIC-SI9945AEY_C3040623.html" (at 189.23 101.6 90)
       (effects (font (size 1.27 1.27)) hide)
     )
@@
       (effects (font (size 1.27 1.27)) hide)
     )
-    (property "lcsc" "https://www.lcsc.com/product-detail/Light-Emitting-Diodes-LED_Foshan-NationStar-Optoelectronics-NCD0805C1_C84257.html" (at 99.06 30.48 90)
+    (property "LCSC" "https://www.lcsc.com/product-detail/Light-Emitting-Diodes-LED_Foshan-NationStar-Optoelectronics-NCD0805C1_C84257.html" (at 99.06 30.48 90)
       (effects (font (size 1.27 1.27)) hide)
     )
@@
       (effects (font (size 1.27 1.27)) hide)
     )
-    (property "lcsc" "https://www.lcsc.com/product-detail/Surge-Suppressors_Analog-Devices-LTC4365ITS8-TRPBF_C514441.html" (at 184.15 120.65 0)
+    (property "LCSC" "https://www.lcsc.com/product-detail/Surge-Suppressors_Analog-Devices-LTC4365ITS8-TRPBF_C514441.html" (at 184.15 120.65 0)
       (effects (font (size 1.27 1.27)) hide)
     )
@@
       (effects (font (size 1.27 1.27)) hide)
     )
-    (property "lcsc" "https://www.lcsc.com/product-detail/Operational-Amplifier_XBLW-LM321DTR-XBLW_C18723612.html" (at 95.25 157.48 0)
+    (property "LCSC" "https://www.lcsc.com/product-detail/Operational-Amplifier_XBLW-LM321DTR-XBLW_C18723612.html" (at 95.25 157.48 0)
       (effects (font (size 1.27 1.27)) hide)
     )
@@
       (effects (font (size 1.27 1.27)) hide)
     )
-    (property "lcsc" "https://www.lcsc.com/product-detail/DC-DC-Converters_Texas-Instruments-LM2596SX-5-0-NOPB_C10002.html" (at 233.68 101.6 0)
+    (property "LCSC" "https://www.lcsc.com/product-detail/DC-DC-Converters_Texas-Instruments-LM2596SX-5-0-NOPB_C10002.html" (at 233.68 101.6 0)
       (effects (font (size 1.27 1.27)) hide)
     )
@@
       (effects (font (size 1.27 1.27)) (justify left) hide)
     )
-    (property "lcsc" "https://www.lcsc.com/product-detail/Bipolar-Transistors-BJT_JSMSEMI-S8050_C916390.html" (at 96.52 69.85 0)
+    (property "LCSC" "https://www.lcsc.com/product-detail/Bipolar-Transistors-BJT_JSMSEMI-S8050_C916390.html" (at 96.52 69.85 0)
       (effects (font (size 1.27 1.27)) hide)
     )
@@
       (effects (font (size 1.27 1.27)) hide)
     )
-    (property "lcsc" "https://www.lcsc.com/product-detail/Schottky-Barrier-Diodes-SBD_LGE-SS53C_C330397.html" (at 125.73 148.59 90)
+    (property "LCSC" "https://www.lcsc.com/product-detail/Schottky-Barrier-Diodes-SBD_LGE-SS53C_C330397.html" (at 125.73 148.59 90)
       (effects (font (size 1.27 1.27)) hide)
     )
@@
       (effects (font (size 1.27 1.27)) hide)
     )
-    (property "lcsc" "https://www.lcsc.com/product-detail/Tantalum-Capacitors_KEMET-T491D227K016AT_C122304.html" (at 267.97 111.76 0)
-      (effects (font (size 1.27 1.27)) hide)
-    )
+    (property "LCSC" "https://www.lcsc.com/product-detail/Tantalum-Capacitors_KEMET-T491D227K016AT_C122304.html" (at 267.97 111.76 0)
+      (effects (font (size 1.27 1.27)) hide)
+    )

Commit message: ...
Parts:
- C1, C2, C3: LCSC (none) -> https://www.lcsc.com/product-detail/Multilayer-Ceramic-Capa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
- R1, R10, R12, R13, R14, R15, R17, R18, R19, R2, R20, R21, R22, R23, R24, R25, R26, R3, R4, R5, R6, R7, R8, R9: LCSC (none) -> https://www.lcsc.com/product-detail/Chip-Resistor-Surface-M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
Changed lines of the file:
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@@
+      (effects (font (size 1.27 1.27)) hide)
+    )
+    (property "LCSC" "https://www.lcsc.com/product-detail/Chip-Resistor-Surface-Mount_UNI-ROYAL-Uniroyal-Elec-0805W8F8202T5E_C17840.html" (at 151.13 124.46 0)
       (effects (font (size 1.27 1.27)) hide)
     )
@@
     )
     (property "Datasheet" "~" (at 96.52 87.63 0)
+      (effects (font (size 1.27 1.27)) hide)
+    )
+    (property "LCSC" "https://www.lcsc.com/product-detail/Multilayer-Ceramic-Capacitors-MLCC-SMD-SMT_CCTC-TCC0805X7R104K500DT_C282732.html" (at 96.52 87.63 0)
       (effects (font (size 1.27 1.27)) hide)
     )
@@
       (effects (font (size 1.27 1.27)) hide)
     )
+    (property "LCSC" "https://www.lcsc.com/product-detail/Chip-Resistor-Surface-Mount_UNI-ROYAL-Uniroyal-Elec-0805W8F1001T5E_C17513.html" (at 96.52 99.06 0)
+      (effects (font (size 1.27 1.27)) hide)
+    )
     (pin "1")
     (pin "2")
@@
       (effects (font (size 1.27 1.27)) hide)
     )
+    (property "LCSC" "https://www.lcsc.com/product-detail/Multilayer-Ceramic-Capacitors-MLCC-SMD-SMT_CCTC-TCC0805X7R104K500DT_C282732.html" (at 139.7 25.4 90)
+      (effects (font (size 1.27 1.27)) hide)
+    )
     (pin "1")
     (pin "2")
@@
       (effects (font (size 1.27 1.27)) hide)
     )
+    (property "LCSC" "https://www.lcsc.com/product-detail/Chip-Resistor-Surface-Mount_UNI-ROYAL-Uniroyal-Elec-0805W8F1001T5E_C17513.html" (at 99.06 39.37 0)
+      (effects (font (size 1.27 1.27)) hide)
+    )
     (pin "1")
     (pin "2")
@@
       (effects (font (size 1.27 1.27)) hide)
     )
+    (property "LCSC" "https://www.lcsc.com/product-detail/Chip-Resistor-Surface-Mount_UNI-ROYAL-Uniroyal-Elec-0805W8F1002T5E_C17414.html" (at 125.73 167.64 0)
+      (effects (font (size 1.27 1.27)) hide)
+    )
     (pin "1")
     (pin "2")
@@
       (effects (font (size 1.27 1.27)) hide)
     )
+    (property "LCSC" "https://www.lcsc.com/product-detail/Chip-Resistor-Surface-Mount_UNI-ROYAL-Uniroyal-Elec-0805W8F1001T5E_C17513.html" (at 88.9 39.37 0)
+      (effects (font (size 1.27 1.27)) hide)
+    )
     (pin "1")
     (pin "2")
@@
     )
     (property "Datasheet" "~" (at 162.56 113.03 0)
+      (effects (font (size 1.27 1.27)) hide)
+    )
+    (property "LCSC" "https://www.lcsc.com/product-detail/Chip-Resistor-Surface-Mount_UNI-ROYAL-Uniroyal-Elec-0805W8F1003T5E_C149504.html" (at 162.56 113.03 90)
       (effects (font (size 1.27 1.27)) hide)
     )
@@
       (effects (font (size 1.27 1.27)) hide)
     )
+    (property "LCSC" "https://www.lcsc.com/product-detail/Chip-Resistor-Surface-Mount_UNI-ROYAL-Uniroyal-Elec-0805W8F4701T5E_C17673.html" (at 151.13 31.75 0)
+      (effects (font (size 1.27 1.27)) hide)
+    )
     (pin "1")
     (pin "2")
@@
     )
     (property "Datasheet" "~" (at 88.9 64.77 0)
+      (effects (font (size 1.27 1.27)) hide)
+    )
+    (property "LCSC" "https://www.lcsc.com/product-detail/Chip-Resistor-Surface-Mount_UNI-ROYAL-Uniroyal-Elec-0805W8F4701T5E_C17673.html" (at 88.9 64.77 0)
       (effects (font (size 1.27 1.27)) hide)
     )
@@
       (effects (font (size 1.27 1.27)) hide)
     )
+    (property "LCSC" "https://www.lcsc.com/product-detail/Chip-Resistor-Surface-Mount_UNI-ROYAL-Uniroyal-Elec-0805W8F0000T5E_C17477.html" (at 99.06 59.69 90)
+      (effects (font (size 1.27 1.27)) hide)
+    )
     (pin "1")
     (pin "2")
@@
     )
     (property "Datasheet" "~" (at 151.13 69.85 0)
+      (effects (font (size 1.27 1.27)) hide)
+    )
+    (property "LCSC" "https://www.lcsc.com/product-detail/Chip-Resistor-Surface-Mount_UNI-ROYAL-Uniroyal-Elec-0805W8F4701T5E_C17673.html" (at 151.13 69.85 0)
       (effects (font (size 1.27 1.27)) hide)
     )
@@
       (effects (font (size 1.27 1.27)) hide)
     )
+    (property "LCSC" "https://www.lcsc.com/product-detail/Chip-Resistor-Surface-Mount_UNI-ROYAL-Uniroyal-Elec-0805W8F4701T5E_C17673.html" (at 157.48 113.03 90)
+      (effects (font (size 1.27 1.27)) hide)
+    )
     (pin "1")
     (pin "2")
@@
       (effects (font (size 1.27 1.27)) hide)
     )
+    (property "LCSC" "https://www.lcsc.com/product-detail/Chip-Resistor-Surface-Mount_UNI-ROYAL-Uniroyal-Elec-0805W8F1002T5E_C17414.html" (at 214.63 40.64 90)
+      (effects (font (size 1.27 1.27)) hide)
+    )
     (pin "1")
     (pin "2")
@@
       (effects (font (size 1.27 1.27)) hide)
     )
+    (property "LCSC" "https://www.lcsc.com/product-detail/Chip-Resistor-Surface-Mount_RALEC-RTH0510R0FTP_C7422239.html" (at 151.13 59.69 0)
+      (effects (font (size 1.27 1.27)) hide)
+    )
     (pin "1")
     (pin "2")
@@
       (effects (font (size 1.27 1.27)) hide)
     )
+    (property "LCSC" "https://www.lcsc.com/product-detail/Multilayer-Ceramic-Capacitors-MLCC-SMD-SMT_CCTC-TCC0805X7R104K500DT_C282732.html" (at 102.87 147.32 90)
+      (effects (font (size 1.27 1.27)) hide)
+    )
     (pin "1")
     (pin "2")
@@
       (effects (font (size 1.27 1.27)) hide)
     )
+    (property "LCSC" "https://www.lcsc.com/product-detail/Chip-Resistor-Surface-Mount_Ever-Ohms-Tech-CRH0805J120RP05Z_C149652.html" (at 151.13 50.8 0)
+      (effects (font (size 1.27 1.27)) hide)
+    )
     (pin "1")
     (pin "2")
@@
     )
     (property "Datasheet" "~" (at 151.13 41.91 0)
+      (effects (font (size 1.27 1.27)) hide)
+    )
+    (property "LCSC" "https://www.lcsc.com/product-detail/Chip-Resistor-Surface-Mount_RALEC-RTH0510R0FTP_C7422239.html" (at 151.13 41.91 0)
       (effects (font (size 1.27 1.27)) hide)
     )
@@
       (effects (font (size 1.27 1.27)) hide)
     )
+    (property "LCSC" "https://www.lcsc.com/product-detail/Chip-Resistor-Surface-Mount_UNI-ROYAL-Uniroyal-Elec-0805W8F8202T5E_C17840.html" (at 151.13 137.16 0)
+      (effects (font (size 1.27 1.27)) hide)
+    )
     (pin "1")
     (pin "2")
@@
       (effects (font (size 1.27 1.27)) hide)
     )
+    (property "LCSC" "https://www.lcsc.com/product-detail/Chip-Resistor-Surface-Mount_UNI-ROYAL-Uniroyal-Elec-0805W8F1002T5E_C17414.html" (at 209.55 40.64 90)
+      (effects (font (size 1.27 1.27)) hide)
+    )
     (pin "1")
     (pin "2")
@@
       (effects (font (size 1.27 1.27)) hide)
     )
+    (property "LCSC" "https://www.lcsc.com/product-detail/Chip-Resistor-Surface-Mount_UNI-ROYAL-Uniroyal-Elec-0805W8F1002T5E_C17414.html" (at 106.68 118.11 0)
+      (effects (font (size 1.27 1.27)) hide)
+    )
     (pin "1")
     (pin "2")
@@
       (effects (font (size 1.27 1.27)) hide)
     )
+    (property "LCSC" "https://www.lcsc.com/product-detail/Chip-Resistor-Surface-Mount_UNI-ROYAL-Uniroyal-Elec-0805W8F1003T5E_C149504.html" (at 157.48 137.16 0)
+      (effects (font (size 1.27 1.27)) hide)
+    )
     (pin "1")
     (pin "2")
@@
     )
     (property "Datasheet" "~" (at 73.66 166.37 0)
+      (effects (font (size 1.27 1.27)) hide)
+    )
+    (property "LCSC" "https://www.lcsc.com/product-detail/Chip-Resistor-Surface-Mount_UNI-ROYAL-Uniroyal-Elec-0805W8F4701T5E_C17673.html" (at 73.66 166.37 0)
       (effects (font (size 1.27 1.27)) hide)
     )
@@
       (effects (font (size 1.27 1.27)) hide)
     )
+    (property "LCSC" "https://www.lcsc.com/product-detail/Chip-Resistor-Surface-Mount_UNI-ROYAL-Uniroyal-Elec-0805W8F4701T5E_C17673.html" (at 118.11 157.48 90)
+      (effects (font (size 1.27 1.27)) hide)
+    )
     (pin "1")
     (pin "2")
@@
       (effects (font (size 1.27 1.27)) hide)
     )
+    (property "LCSC" "https://www.lcsc.com/product-detail/Chip-Resistor-Surface-Mount_UNI-ROYAL-Uniroyal-Elec-0805W8F1002T5E_C17414.html" (at 109.22 39.37 0)
+      (effects (font (size 1.27 1.27)) hide)
+    )
     (pin "1")
     (pin "2")
@@
       (effects (font (size 1.27 1.27)) hide)
     )
+    (property "LCSC" "https://www.lcsc.com/product-detail/Chip-Resistor-Surface-Mount_UNI-ROYAL-Uniroyal-Elec-0805W8F1001T5E_C17513.html" (at 139.7 113.03 0)
+      (effects (font (size 1.27 1.27)) hide)
+    )
     (pin "1")
     (pin "2")
@@
       (effects (font (size 1.27 1.27)) hide)
     )
+    (property "LCSC" "https://www.lcsc.com/product-detail/Chip-Resistor-Surface-Mount_FOJAN-FRC0805J275-TS_C2933540.html" (at 151.13 113.03 90)
+      (effects (font (size 1.27 1.27)) hide)
+    )
