File: MasterShield.kicad_sch (KiCad schematic)
At the start: 66 parts, among them J1 CONTROL/SERIAL, J2 MISC, J3 ADC/SENSE, J4 POWER, J5 RS485 A, J6 EXTRA POWER, J7 BATT, J8 RS485 B, Q1 S8050, Q2 Si9945AEY-T1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

Commit message: ...
Parts:
- C1, C2, C3: LCSC https://www.lcsc.com/product-detail/Multilayer-Ceramic-Capa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 -> C282732
- C4: LCSC https://www.lcsc.com/product-detail/Aluminum-Electrolytic-C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 -> C7461236
- C5: LCSC https://www.lcsc.com/product-detail/Tantalum-Capacitors_KEM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 -> C122304
- D1, D2: LCSC https://www.lcsc.com/product-detail/Light-Emitting-Diodes-L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 -> C84257
- D3, D5: LCSC https://www.lcsc.com/product-detail/Schottky-Barrier-Diodes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 -> C330397
- D4: LCSC https://www.lcsc.com/product-detail/Zener-Diodes_Nexperia-P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 -> C85383
- D6: LCSC https://www.lcsc.com/product-detail/Light-Emitting-Diodes-s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 -> C434431
- L1: LCSC https://www.lcsc.com/product-detail/Power-Inductors_cjiang-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 -> C177245
- Q1, Q3: LCSC https://www.lcsc.com/product-detail/Bipolar-Transistors-BJT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 -> C916390
- Q2: LCSC https://www.lcsc.com/product-detail/MOSFETs_TECH-PUBLIC-SI9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 -> C3040623
- R1, R17, R20, R26, R3, R8: LCSC https://www.lcsc.com/product-detail/Chip-Resistor-Surface-M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 -> C17673
- R10, R12, R13, R14, R21: LCSC https://www.lcsc.com/product-detail/Chip-Resistor-Surface-M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 -> C17414
- R15, R24, R4, R9: LCSC https://www.lcsc.com/product-detail/Chip-Resistor-Surface-M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 -> C17513
- R18: LCSC https://www.lcsc.com/product-detail/Chip-Resistor-Surface-M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 -> C2933540
- R19, R22: LCSC https://www.lcsc.com/product-detail/Chip-Resistor-Surface-M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 -> C17840
- R2: LCSC https://www.lcsc.com/product-detail/Chip-Resistor-Surface-M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 -> C17477
- R23, R25: LCSC https://www.lcsc.com/product-detail/Chip-Resistor-Surface-M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 -> C149504
- R5, R7: LCSC https://www.lcsc.com/product-detail/Chip-Resistor-Surface-M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 -> C7422239
- R6: LCSC https://www.lcsc.com/product-detail/Chip-Resistor-Surface-M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 -> C149652
- U1: LCSC https://www.lcsc.com/product-detail/RS-span-style-backgroun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 -> C481667
- U2: LCSC https://www.lcsc.com/product-detail/Power-Distribution-Swit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 -> C82656
- U3: LCSC https://www.lcsc.com/product-detail/Gates_Nexperia-74LVC1G0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 -> C12512
- U4: LCSC https://www.lcsc.com/product-detail/Operational-Amplifier_X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 -> C18723612
- U5: LCSC https://www.lcsc.com/product-detail/DC-DC-Converters_Texas-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 -> C10002
- U6: LCSC https://www.lcsc.com/product-detail/Surge-Suppressors_Analo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 -> C514441

Commit message: ...
Parts:
- removed D5: SS53C, Diode_SMD:D_SOD-323_HandSoldering, symbol Diode:1N5817
- added D5: BZT52C3V3S, Diode_SMD:D_SOD-323_HandSoldering, symbol Device:D_Zener
- added D7: SS54, Diode_SMD:D_SMC_Handsoldering, symbol Diode:1N5817
- added J9: BYPASS, Connector_PinHeader_2.54mm:PinHeader_1x02_P2.54mm_Vertical, symbol Connector:Conn_01x02_Pin
- D3: value SS53C -> SS54; footprint Diode_SMD:D_SOD-323_HandSoldering -> Diode_SMD:D_SMC_Handsoldering; LCSC C330397 -> C22452
- R6: LCSC C149652 -> C844392
Connections:
- net +5V: now also D7.2 (A), J9.1 (Pin_1)
- net AD0: now also D5.1 (K)
- net GND: now also D5.2 (A)
- net VDD (5V): now also D7.1 (K), J9.2 (Pin_2)
Other:
- moved on the sheet: C5, D3

Commit message: ...
Parts:
- D3, D7: footprint Diode_SMD:D_SMC_Handsoldering -> Diode_SMD:D_SMA_Handsoldering
Changed lines of the file:
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@@
       (effects (font (size 1.27 1.27)) (justify left))
     )
-    (property "Footprint" "Diode_SMD:D_SMC_Handsoldering" (at 241.935 113.03 0)
+    (property "Footprint" "Diode_SMD:D_SMA_Handsoldering" (at 241.935 113.03 0)
       (effects (font (size 1.27 1.27)) hide)
     )
@@
       (effects (font (size 1.27 1.27)))
     )
-    (property "Footprint" "Diode_SMD:D_SMC_Handsoldering" (at 66.04 122.555 0)
-      (effects (font (size 1.27 1.27)) hide)
-    )
+    (property "Footprint" "Diode_SMD:D_SMA_Handsoldering" (at 66.04 122.555 0)
+      (effects (font (size 1.27 1.27)) hide)
+    )

Commit message: ...
Parts:
- removed D5: BZT52C3V3S, Diode_SMD:D_SOD-323_HandSoldering, symbol Device:D_Zener
- D4: value 10V -> BZT52C9V1; footprint Diode_SMD:D_SOD-323_HandSoldering -> Diode_SMD:D_SOD-123; LCSC C85383 -> C5270765; mouser https://eu.mouser.com/ProductDetail/Nexperia/PDZ10B115?qs=L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 -> (none); part PDZ10B -> (none)
- R17: value 4.7k -> 5.1K
Connections:
- net +12V: now also C3.1, U4.5 (V+); no longer D4.1 (K)
- net +5V: no longer C3.1, U4.5 (V+)
- net +BATT: now also D4.1 (K)
Other:
- moved on the sheet: TP10

Commit message: ...
Parts:
- removed C1: 0.1uF, Capacitor_SMD:C_0805_2012Metric, symbol Device:C
- removed R11, R16: 0R, Resistor_SMD:R_0805_2012Metric, symbol Device:R
- removed R14: 10K, Resistor_SMD:R_0805_2012Metric, symbol Device:R
- removed R15: 1K, Resistor_SMD:R_0805_2012Metric, symbol Device:R
- removed TP5: UV, TestPoint:TestPoint_Pad_D2.0mm, symbol Connector:TestPoint
- removed TP6: OV, TestPoint:TestPoint_Pad_D2.0mm, symbol Connector:TestPoint
- removed U3: 74LVC1G08GW, Package_TO_SOT_SMD:SOT-353_SC-70-5, symbol 74xGxx:74AUC1G08
- added C1: 680uF, Capacitor_SMD:CP_Elec_10x10.5, symbol Device:C_Polarized
- added C6: 0.1uF, Capacitor_SMD:C_0805_2012Metric, symbol Device:C
- added D5: TXD, LED_SMD:LED_0805_2012Metric, symbol Device:LED
- added SW1: SW_Push_DPDT, Button_Switch_SMD:Nidec_Copal_SH-7010A, symbol Switch:SW_Push_DPDT
- R2: value 0R -> 1K; LCSC C17477 -> C17513
- TP1: value RO -> DIR
- TP2: value DI -> FGO
- TP3: value ~{RE} -> UV
- TP4: value DE -> OV
Connections:
- net +BATT: now also R2.1, C1.1
- net AD0: now also TP2.1
- net GND: now also C1.2, C6.1, D5.1 (K)
- net P0.00: no longer TP1.1
- net P0.01: no longer TP2.1
- net P0.02: now also SW1.1 (A), SW1.4 (A)
- net at R18.2, R19.1, U6.2 (UV): now also TP3.1, C6.2
- net at R19.2, R22.1, U6.3 (OV): now also TP4.1
- net at R10.2, U1.2 (~{RE}): now also TP1.1, U1.3 (DE), SW1.2 (B), SW1.5 (B); no longer R2.2, TP3.1
- net at Q1.3 (C): now also SW1.3 (C), SW1.6 (C); no longer R2.1
- new net: D5.2 (A), R2.2
Other:
- moved on the sheet: D1, D6, Q1, R1, R10, R18, R19, R22, R24, R9
