File: MasterShield.kicad_pcb (KiCad board)
At the start: 4 copper layers, 63.5 x 91.4 mm, 70 parts, among them J1 CONTROL/SERIAL, J2 MISC, J3 ADC/SENSE, J4 POWER, J5 RS485 B, J6 EXTRA POWER, J7 BATT, J8 RS485 A, Q1 S8050, Q2 Si9945AEY-T1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

Commit message: ...
Parts:
- removed REF** (x4): MountingHole_2.5mm_Pad, MountingHole:MountingHole_2.5mm_Pad
- J7: value BATT -> BATTERY
Other:
- board text added: "+"
- board text added: "-"
- board text added: "A"
- board text added: "B"
- board text added: "OUT1"
- board text added: "OUT2"
- board text added: "OUT3"
- board text added: "OUT4"
Changed lines of the file:
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@@
     (property "ki_keywords" "screw terminal")
     (attr through_hole)
-    (fp_text reference "J5" (at 0.7314 4.7244 180) (layer "F.SilkS")
+    (fp_text reference "J5" (at 5.278 2.921 180) (layer "F.SilkS")
         (effects (font (size 1 1) (thickness 0.15)))
     )
-    (fp_text value "RS485 B" (at 5.4558 4.6736 180) (layer "F.SilkS")
+    (fp_text value "RS485 B" (at -3.5104 0.4064 270) (layer "F.SilkS")
         (effects (font (size 1 1) (thickness 0.15)))
     )
@@
     )
   )
-  (footprint "MountingHole:MountingHole_2.5mm_Pad" (layer "F.Cu")
-    (at 200.66 132.08)
-    (descr "Mounting Hole 2.5mm")
-    (tags "mounting hole 2.5mm")
-    (attr exclude_from_pos_files exclude_from_bom)
-    (fp_text reference "REF**" (at 0 -3.5) (layer "F.SilkS") hide
-        (effects (font (size 1 1) (thickness 0.15)))
-    )
-    (fp_text value "MountingHole_2.5mm_Pad" (at 0 3.5) (layer "F.Fab") hide
-        (effects (font (size 1 1) (thickness 0.15)))
-    )
-    (fp_text user "${REFERENCE}" (at 0 0) (layer "F.Fab")
-        (effects (font (size 1 1) (thickness 0.15)))
-    )
-    (fp_circle (center 0 0) (end 2.5 0)
-      (stroke (width 0.15) (type solid)) (fill none) (layer "Cmts.User"))
-    (fp_circle (center 0 0) (end 2.75 0)
-      (stroke (width 0.05) (type solid)) (fill none) (layer "F.CrtYd"))
-    (pad "1" thru_hole circle (at 0 0) (size 5 5) (drill 2.5) (layers "*.Cu" "*.Mask"))
-  )
   (footprint "TestPoint:TestPoint_Pad_D2.0mm" (layer "F.Cu")
     (at 210.185 93.726 -90)
@@
     )
   )
-  (footprint "MountingHole:MountingHole_2.5mm_Pad" (layer "F.Cu")
-    (at 254 132.08)
-    (descr "Mounting Hole 2.5mm")
-    (tags "mounting hole 2.5mm")
-    (attr exclude_from_pos_files exclude_from_bom)
-    (fp_text reference "REF**" (at 0 -3.5) (layer "F.SilkS") hide
-        (effects (font (size 1 1) (thickness 0.15)))
-    )
-    (fp_text value "MountingHole_2.5mm_Pad" (at -10.16 3.5 180) (layer "F.Fab") hide
-        (effects (font (size 1 1) (thickness 0.15)))
-    )
-    (fp_text user "${REFERENCE}" (at 0 0) (layer "F.Fab")
-        (effects (font (size 1 1) (thickness 0.15)))
-    )
-    (fp_circle (center 0 0) (end 2.5 0)
-      (stroke (width 0.15) (type solid)) (fill none) (layer "Cmts.User"))
-    (fp_circle (center 0 0) (end 2.75 0)
-      (stroke (width 0.05) (type solid)) (fill none) (layer "F.CrtYd"))
-    (pad "1" thru_hole circle (at 0 0) (size 5 5) (drill 2.5) (layers "*.Cu" "*.Mask"))
-  )
   (footprint "Resistor_SMD:R_0805_2012Metric" (layer "F.Cu")
     (at 224.6395 91.44 180)
@@
         (effects (font (size 1 1) (thickness 0.15)))
     )
-    (fp_text value "RXD" (at 2.4915 0 180) (layer "F.SilkS")
+    (fp_text value "RXD" (at 3.2027 0.0762 180) (layer "F.SilkS")
         (effects (font (size 1 1) (thickness 0.15)))
     )
@@
         (effects (font (size 1 1) (thickness 0.15)))
     )
-    (fp_text value "RS485 A" (at 5.25 4.66) (layer "F.SilkS")
+    (fp_text value "RS485 A" (at 14.0104 0.4572 90) (layer "F.SilkS")
         (effects (font (size 1 1) (thickness 0.15)))
     )
@@
     )
   )
-  (footprint "MountingHole:MountingHole_2.5mm_Pad" (layer "F.Cu")
-    (at 200.66 50.8)
-    (descr "Mounting Hole 2.5mm")
-    (tags "mounting hole 2.5mm")
-    (attr exclude_from_pos_files exclude_from_bom)
-    (fp_text reference "REF**" (at 0 -3.5) (layer "F.SilkS") hide
-        (effects (font (size 1 1) (thickness 0.15)))
-    )
-    (fp_text value "MountingHole_2.5mm_Pad" (at 0 3.5) (layer "F.Fab") hide
-        (effects (font (size 1 1) (thickness 0.15)))
-    )
-    (fp_text user "${REFERENCE}" (at 0 0) (layer "F.Fab")
-        (effects (font (size 1 1) (thickness 0.15)))
-    )
-    (fp_circle (center 0 0) (end 2.5 0)
-      (stroke (width 0.15) (type solid)) (fill none) (layer "Cmts.User"))
-    (fp_circle (center 0 0) (end 2.75 0)
-      (stroke (width 0.05) (type solid)) (fill none) (layer "F.CrtYd"))
-    (pad "1" thru_hole circle (at 0 0) (size 5 5) (drill 2.5) (layers "*.Cu" "*.Mask"))
-  )
   (footprint "TerminalBlock_4Ucon:TerminalBlock_4Ucon_1x04_P3.50mm_Horizontal" (layer "F.Cu")
     (at 205.232 108.077 -90)
@@
         (effects (font (size 1 1) (thickness 0.15)))
     )
-    (fp_text value "BATT" (at 5.25 4.66 90) (layer "F.SilkS")
+    (fp_text value "BATTERY" (at 13.97 -0.0254 180) (layer "F.SilkS")
         (effects (font (size 1 1) (thickness 0.15)))
     )
@@
         (effects (font (size 1 1) (thickness 0.15)))
     )
-    (fp_text value "TXD" (at 2.5885 0 180) (layer "F.SilkS")
+    (fp_text value "TXD" (at 3.2027 0.0762) (layer "F.SilkS")
         (effects (font (size 1 1) (thickness 0.15)))
     )
@@
         (effects (font (size 1 1) (thickness 0.15)))
     )
-    (fp_text value "EXTRA POWER" (at 5.25 4.66 90) (layer "F.SilkS")
+    (fp_text value "EXTRA POWER" (at -3.597 -0.1016 180) (layer "F.SilkS")
         (effects (font (size 1 1) (thickness 0.15)))
     )
@@
     )
   )
-  (footprint "MountingHole:MountingHole_2.5mm_Pad" (layer "F.Cu")
-    (at 254 50.8)
-    (descr "Mounting Hole 2.5mm")
-    (tags "mounting hole 2.5mm")
-    (attr exclude_from_pos_files exclude_from_bom)
-    (fp_text reference "REF**" (at 0 -3.5) (layer "F.SilkS") hide
-        (effects (font (size 1 1) (thickness 0.15)))
-    )
-    (fp_text value "MountingHole_2.5mm_Pad" (at 0 3.5) (layer "F.Fab") hide
-        (effects (font (size 1 1) (thickness 0.15)))
-    )
-    (fp_text user "${REFERENCE}" (at 0 0) (layer "F.Fab")
-        (effects (font (size 1 1) (thickness 0.15)))
-    )
-    (fp_circle (center 0 0) (end 2.5 0)
-      (stroke (width 0.15) (type solid)) (fill none) (layer "Cmts.User"))
-    (fp_circle (center 0 0) (end 2.75 0)
-      (stroke (width 0.05) (type solid)) (fill none) (layer "F.CrtYd"))
-    (pad "1" thru_hole circle (at 0 0) (size 5 5) (drill 2.5) (layers "*.Cu" "*.Mask"))
-  )
   (footprint "Package_SO:SOIC-8_3.9x4.9mm_P1.27mm" (layer "F.Cu")
     (at 233.553 72.263 90)
@@
   (gr_arc (start 256.54 45.72) (mid 258.336051 46.463949) (end 259.08 48.26)
     (stroke (width 0.1) (type default)) (layer "Edge.Cuts"))
+  (gr_text "+" (at 201.171972 119.761) (layer "F.SilkS")
+    (effects (font (size 1.5 1.5) (thickness 0.3) bold) (justify left bottom mirror))
+  )
+  (gr_text "-" (at 240.495714 53.4162 180) (layer "F.SilkS")
+    (effects (font (size 1.5 1.5) (thickness 0.3) bold) (justify left bottom mirror))
+  )
+  (gr_text "-" (at 200.9394 110.411247 90) (layer "F.SilkS")
+    (effects (font (size 1.5 1.5) (thickness 0.3) bold) (justify left bottom mirror))
+  )
+  (gr_text "+" (at 201.171972 116.110694) (layer "F.SilkS")
+    (effects (font (size 1.5 1.5) (thickness 0.3) bold) (justify left bottom mirror))
+  )
+  (gr_text "+" (at 245.8974 54.991) (layer "F.SilkS")
+    (effects (font (size 1.5 1.5) (thickness 0.3) bold) (justify left bottom mirror))
+  )
+  (gr_text "B" (at 235.6358 54.9148) (layer "F.SilkS")
+    (effects (font (size 1.5 1.5) (thickness 0.3) bold) (justify left bottom mirror))
+  )
+  (gr_text "-" (at 251.46 110.6932 180) (layer "F.SilkS")
+    (effects (font (size 5 5) (thickness 0.15)) (justify left bottom mirror))
+  )
+  (gr_text "-" (at 255.545428 117.5766 90) (layer "F.SilkS")
+    (effects (font (size 1.5 1.5) (thickness 0.3) bold) (justify left bottom mirror))
+  )
+  (gr_text "+" (at 255.778 115.8494) (layer "F.SilkS")
+    (effects (font (size 1.5 1.5) (thickness 0.3) bold) (justify left bottom mirror))
+  )
+  (gr_text "-" (at 214.460714 53.3146 180) (layer "F.SilkS")
+    (effects (font (size 1.5 1.5) (thickness 0.3) bold) (justify left bottom mirror))
+  )
+  (gr_text "A\n" (at 211.328 52.8828 180) (layer "F.SilkS")
+    (effects (font (size 1.5 1.5) (thickness 0.3) bold) (justify left bottom mirror))
+  )
+  (gr_text "OUT3" (at 217.2208 52.959 180) (layer "F.SilkS")
+    (effects (font (size 0.5 0.5) (thickness 0.125)))
+  )
+  (gr_text "OUT2" (at 256.0828 109.601 90) (layer "F.SilkS")
+    (effects (font (size 0.5 0.5) (thickness 0.125)))
+  )
+  (gr_text "OUT4" (at 243.1542 53.1622 180) (layer "F.SilkS")
+    (effects (font (size 0.5 0.5) (thickness 0.125)))
+  )
+  (gr_text "-" (at 200.9394 107.1118 90) (layer "F.SilkS")
+    (effects (font (size 1.5 1.5) (thickness 0.3) bold) (justify left bottom mirror))
+  )
+  (gr_text "B" (at 209.423 54.8894) (layer "F.SilkS")
+    (effects (font (size 1.5 1.5) (thickness 0.3) bold) (justify left bottom mirror))
+  )
+  (gr_text "+" (at 255.778 112.0394) (layer "F.SilkS")
+    (effects (font (size 1.5 1.5) (thickness 0.3) bold) (justify left bottom mirror))
+  )
+  (gr_text "+" (at 219.8624 54.8894) (layer "F.SilkS")
+    (effects (font (size 1.5 1.5) (thickness 0.3) bold) (justify left bottom mirror))
+  )
+  (gr_text "-" (at 255.545428 106.850506 90) (layer "F.SilkS")
+    (effects (font (size 1.5 1.5) (thickness 0.3) bold) (justify left bottom mirror))
+  )
+  (gr_text "-" (at 196.8754 110.8964 180) (layer "F.SilkS")
+    (effects (font (size 5 5) (thickness 0.15)) (justify left bottom mirror))
+  )
+  (gr_text "OUT1" (at 255.9558 116.9416 90) (layer "F.SilkS")
+    (effects (font (size 0.5 0.5) (thickness 0.125)))
+  )
+  (gr_text "A\n" (at 237.363 52.9844 180) (layer "F.SilkS")
+    (effects (font (size 1.5 1.5) (thickness 0.3) bold) (justify left bottom mirror))
+  )
   (segment (start 227.203 68.58) (end 228.216 68.58) (width 0.25) (layer "F.Cu") (net 1))
   (segment (start 224.917 57.942) (end 226.598 57.942) (width 0.3) (layer "F.Cu") (net 1))
