File: MasterShield.kicad_pcb (KiCad board)
At the start: 4 copper layers, 63.5 x 91.4 mm, 66 parts, among them J1 CONTROL/SERIAL, J2 MISC, J3 ADC/SENSE, J4 POWER, J5 RS485 B, J6 EXTRA POWER, J7 BATTERY, J8 RS485 A, Q1 S8050, Q2 Si9945AEY-T1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

Commit message: ...
Parts:
- J5: value RS485 B -> RS485 A
- J7: value BATTERY -> BATT
- J8: value RS485 A -> RS485 B

Commit message: ...
Parts:
- added D7: SS54, Diode_SMD:D_SMC_Handsoldering, F.Cu at (213.9, 111.4)
- added J9: BYPASS, Connector_PinHeader_2.54mm:PinHeader_1x02_P2.54mm_Vertical, F.Cu at (215.2, 121.6)
- D3: value SS53C -> SS54; footprint Diode_SMD:D_SOD-323_HandSoldering -> Diode_SMD:D_SMC_Handsoldering
- D5: value SS53C -> BZT52C3V3S
- moved D3 20.7 mm to (241.4, 119.8), turned to -90 degrees
- moved D4 1.34 mm to (208.2, 74.5)
- moved D5 0.47 mm to (207.1, 69.0), turned to -90 degrees
Connections:
- D5 pad 1: +3.3V -> /AD0
- D5 pad 2: /AD0 -> GND
Routing:
- net /VDD (5V): track 0.00 -> 53.2 mm, vias 0 -> 3
- net +5V: track 164.8 -> 182.2 mm, vias 11 -> 14
- net GND: track 340.0 -> 352.5 mm, vias 38 -> 40
- net Net-(D3-K): track 23.0 -> 31.7 mm
- net +3.3V: track 58.1 -> 51.9 mm
- net /AD0: track 35.4 -> 41.0 mm
- net Net-(Q3-C): track 23.9 -> 25.7 mm
- net Net-(D4-A): track 25.7 -> 24.4 mm
- net /P0.05: track 6.13 -> 5.45 mm
- net /P0.01: track 82.9 -> 82.3 mm

Commit message: ...
Parts:
- D3, D7: footprint Diode_SMD:D_SMC_Handsoldering -> Diode_SMD:D_SMA_Handsoldering
Routing:
- net Net-(D3-K): track 31.7 -> 29.0 mm
- net /VDD (5V): track 53.2 -> 55.3 mm, vias 3 -> 2
- net +5V: track 182.2 -> 183.9 mm, vias 14 -> 13
- net GND: track 352.5 -> 352.3 mm, vias 40 -> 39

Commit message: ...
Parts:
- removed D5: BZT52C3V3S, Diode_SMD:D_SOD-323_HandSoldering
- D4: value 10V -> BZT52C9V1; footprint Diode_SMD:D_SOD-323_HandSoldering -> Diode_SMD:D_SOD-123
- R17: value 4.7k -> 5.1K
Connections:
- C3 pad 1: +5V -> +12V
- D4 pad 1: +12V -> +BATT
- U4 pad 5: +5V -> +12V
Routing:
- net +BATT: track 82.2 -> 111.8 mm, vias 0 -> 2
- net +5V: track 183.9 -> 171.9 mm, vias 13 -> 12
- net /AD0: track 41.0 -> 39.6 mm
- net Net-(D4-A): track 24.4 -> 25.0 mm
